File: V1/ESP-relay-32ch-V1-expanders.kicad_sch (KiCad schematic)
At the start: 8 parts, among them U25 MCP23017_SS, U26 MCP23017_SS, U27 MCP23017_SS

Commit message: Dev
Parts:
- U25, U26, U27: Case (none) -> SSOP-28-5.3; JLCPCB BOM (none) -> 1; LCSC Part # (none) -> C558584; Mfr (none) -> Microchip; Mfr PN (none) -> MCP23017T-E/SS; Vendor (none) -> JLCPCB; Vendor PN (none) -> C558584
Changed lines of the file:
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@@
       (effects (font (size 1.27 1.27)) (justify left) hide)
     )
-    (property "Datasheet" "http://ww1.microchip.com/downloads/en/DeviceDoc/20001952C.pdf" (at 63.5 129.54 0)
+    (property "Datasheet" "" (at 63.5 129.54 0)
       (effects (font (size 1.27 1.27)) (justify left) hide)
+    )
+    (property "JLCPCB BOM" "1" (at 58.42 101.6 0)
+      (effects (font (size 1.27 1.27)) hide)
+    )
+    (property "Case" "SSOP-28-5.3" (at 58.42 101.6 0)
+      (effects (font (size 1.27 1.27)) hide)
+    )
+    (property "LCSC Part #" "C558584" (at 58.42 101.6 0)
+      (effects (font (size 1.27 1.27)) hide)
+    )
+    (property "Mfr" "Microchip" (at 58.42 101.6 0)
+      (effects (font (size 1.27 1.27)) hide)
+    )
+    (property "Mfr PN" "MCP23017T-E/SS" (at 58.42 101.6 0)
+      (effects (font (size 1.27 1.27)) hide)
+    )
+    (property "Technology" "~" (at 58.42 101.6 0)
+      (effects (font (size 1.27 1.27)) hide)
+    )
+    (property "Vendor" "JLCPCB" (at 58.42 101.6 0)
+      (effects (font (size 1.27 1.27)) hide)
+    )
+    (property "Vendor PN" "C558584" (at 58.42 101.6 0)
+      (effects (font (size 1.27 1.27)) hide)
     )
     (pin "1")
@@
       (effects (font (size 1.27 1.27)) (justify left) hide)
     )
-    (property "Datasheet" "http://ww1.microchip.com/downloads/en/DeviceDoc/20001952C.pdf" (at 124.46 129.54 0)
+    (property "Datasheet" "" (at 124.46 129.54 0)
       (effects (font (size 1.27 1.27)) (justify left) hide)
+    )
+    (property "JLCPCB BOM" "1" (at 119.38 101.6 0)
+      (effects (font (size 1.27 1.27)) hide)
+    )
+    (property "Case" "SSOP-28-5.3" (at 119.38 101.6 0)
+      (effects (font (size 1.27 1.27)) hide)
+    )
+    (property "LCSC Part #" "C558584" (at 119.38 101.6 0)
+      (effects (font (size 1.27 1.27)) hide)
+    )
+    (property "Mfr" "Microchip" (at 119.38 101.6 0)
+      (effects (font (size 1.27 1.27)) hide)
+    )
+    (property "Mfr PN" "MCP23017T-E/SS" (at 119.38 101.6 0)
+      (effects (font (size 1.27 1.27)) hide)
+    )
+    (property "Technology" "~" (at 119.38 101.6 0)
+      (effects (font (size 1.27 1.27)) hide)
+    )
+    (property "Vendor" "JLCPCB" (at 119.38 101.6 0)
+      (effects (font (size 1.27 1.27)) hide)
+    )
+    (property "Vendor PN" "C558584" (at 119.38 101.6 0)
+      (effects (font (size 1.27 1.27)) hide)
     )
     (pin "1")
@@
       (effects (font (size 1.27 1.27)) (justify left) hide)
     )
-    (property "Datasheet" "http://ww1.microchip.com/downloads/en/DeviceDoc/20001952C.pdf" (at 185.42 129.54 0)
+    (property "Datasheet" "" (at 185.42 129.54 0)
       (effects (font (size 1.27 1.27)) (justify left) hide)
+    )
+    (property "JLCPCB BOM" "1" (at 180.34 101.6 0)
+      (effects (font (size 1.27 1.27)) hide)
+    )
+    (property "Case" "SSOP-28-5.3" (at 180.34 101.6 0)
+      (effects (font (size 1.27 1.27)) hide)
+    )
+    (property "LCSC Part #" "C558584" (at 180.34 101.6 0)
+      (effects (font (size 1.27 1.27)) hide)
+    )
+    (property "Mfr" "Microchip" (at 180.34 101.6 0)
+      (effects (font (size 1.27 1.27)) hide)
+    )
+    (property "Mfr PN" "MCP23017T-E/SS" (at 180.34 101.6 0)
+      (effects (font (size 1.27 1.27)) hide)
+    )
+    (property "Technology" "~" (at 180.34 101.6 0)
+      (effects (font (size 1.27 1.27)) hide)
+    )
+    (property "Vendor" "JLCPCB" (at 180.34 101.6 0)
+      (effects (font (size 1.27 1.27)) hide)
+    )
+    (property "Vendor PN" "C558584" (at 180.34 101.6 0)
+      (effects (font (size 1.27 1.27)) hide)
     )
     (pin "1")
@@
       (effects (font (size 1.27 1.27)) (justify left) hide)
     )
-    (property "Datasheet" "http://ww1.microchip.com/downloads/en/DeviceDoc/20001952C.pdf" (at 246.38 129.54 0)
+    (property "Datasheet" "" (at 246.38 129.54 0)
       (effects (font (size 1.27 1.27)) (justify left) hide)
     )
-    (pin "1")
+    (property "JLCPCB BOM" "1" (at 241.3 101.6 0)
+      (effects (font (size 1.27 1.27)) hide)
+    )
+    (property "Case" "SSOP-28-5.3" (at 241.3 101.6 0)
+      (effects (font (size 1.27 1.27)) hide)
+    )
+    (property "LCSC Part #" "C558584" (at 241.3 101.6 0)
+      (effects (font (size 1.27 1.27)) hide)
+    )
+    (property "Mfr" "Microchip" (at 241.3 101.6 0)
+      (effects (font (size 1.27 1.27)) hide)
+    )
+    (property "Mfr PN" "MCP23017T-E/SS" (at 241.3 101.6 0)
+      (effects (font (size 1.27 1.27)) hide)
+    )
+    (property "Technology" "~" (at 241.3 101.6 0)
+      (effects (font (size 1.27 1.27)) hide)
+    )
+    (property "Vendor" "JLCPCB" (at 241.3 101.6 0)
+      (effects (font (size 1.27 1.27)) hide)
+    )
+    (property "Vendor PN" "C558584" (at 241.3 101.6 0)
+      (effects (font (size 1.27 1.27)) hide)
+    )
+    (pin "1")
