File: V1/ESP-relay-32ch-V1-inputs-1.kicad_sch (KiCad schematic)
At the start: 112 parts, among them U10 LTV-817S, U11 LTV-817S, U12 LTV-817S, U13 LTV-817S, U14 LTV-817S, U15 LTV-817S, U16 LTV-817S, U17 LTV-817S, U18 LTV-817S, U19 LTV-817S, U20 LTV-817S, U21 LTV-817S, U22 LTV-817S, U23 LTV-817S, U24 LTV-817S, U25 LTV-817S

Commit message: Dev
Parts:
- U10: renamed from U12; value LTV-817S -> OR-3H4-4; footprint Tales:SMDIP-4_W9.53mm -> Package_SO:SOP-16_4.4x10.4mm_P1.27mm; symbol Isolator:LTV-817S -> Tales:OR-3H4-4; Case SMDIP-4 -> SOP-16-4.4; LCSC Part # C109227 -> C2838167; Mfr Lite-On -> Orient; Mfr PN LTV-817S-TA1-C -> OR-3H4-4GB-TA1-GK; Vendor PN C109227 -> C2838167
- U10: value LTV-817S -> OR-3H4-4; footprint Tales:SMDIP-4_W9.53mm -> Package_SO:SOP-16_4.4x10.4mm_P1.27mm; symbol Isolator:LTV-817S -> Tales:OR-3H4-4; Case SMDIP-4 -> SOP-16-4.4; LCSC Part # C109227 -> C2838167; Mfr Lite-On -> Orient; Mfr PN LTV-817S-TA1-C -> OR-3H4-4GB-TA1-GK; Vendor PN C109227 -> C2838167
- U10: renamed from U11; value LTV-817S -> OR-3H4-4; footprint Tales:SMDIP-4_W9.53mm -> Package_SO:SOP-16_4.4x10.4mm_P1.27mm; symbol Isolator:LTV-817S -> Tales:OR-3H4-4; Case SMDIP-4 -> SOP-16-4.4; LCSC Part # C109227 -> C2838167; Mfr Lite-On -> Orient; Mfr PN LTV-817S-TA1-C -> OR-3H4-4GB-TA1-GK; Vendor PN C109227 -> C2838167
- U10: renamed from U13; value LTV-817S -> OR-3H4-4; footprint Tales:SMDIP-4_W9.53mm -> Package_SO:SOP-16_4.4x10.4mm_P1.27mm; symbol Isolator:LTV-817S -> Tales:OR-3H4-4; Case SMDIP-4 -> SOP-16-4.4; LCSC Part # C109227 -> C2838167; Mfr Lite-On -> Orient; Mfr PN LTV-817S-TA1-C -> OR-3H4-4GB-TA1-GK; Vendor PN C109227 -> C2838167
- U11: renamed from U14; value LTV-817S -> OR-3H4-4; footprint Tales:SMDIP-4_W9.53mm -> Package_SO:SOP-16_4.4x10.4mm_P1.27mm; symbol Isolator:LTV-817S -> Tales:OR-3H4-4; Case SMDIP-4 -> SOP-16-4.4; LCSC Part # C109227 -> C2838167; Mfr Lite-On -> Orient; Mfr PN LTV-817S-TA1-C -> OR-3H4-4GB-TA1-GK; Vendor PN C109227 -> C2838167
- U11: renamed from U16; value LTV-817S -> OR-3H4-4; footprint Tales:SMDIP-4_W9.53mm -> Package_SO:SOP-16_4.4x10.4mm_P1.27mm; symbol Isolator:LTV-817S -> Tales:OR-3H4-4; Case SMDIP-4 -> SOP-16-4.4; LCSC Part # C109227 -> C2838167; Mfr Lite-On -> Orient; Mfr PN LTV-817S-TA1-C -> OR-3H4-4GB-TA1-GK; Vendor PN C109227 -> C2838167
- U11: renamed from U17; value LTV-817S -> OR-3H4-4; footprint Tales:SMDIP-4_W9.53mm -> Package_SO:SOP-16_4.4x10.4mm_P1.27mm; symbol Isolator:LTV-817S -> Tales:OR-3H4-4; Case SMDIP-4 -> SOP-16-4.4; LCSC Part # C109227 -> C2838167; Mfr Lite-On -> Orient; Mfr PN LTV-817S-TA1-C -> OR-3H4-4GB-TA1-GK; Vendor PN C109227 -> C2838167
- U11: renamed from U15; value LTV-817S -> OR-3H4-4; footprint Tales:SMDIP-4_W9.53mm -> Package_SO:SOP-16_4.4x10.4mm_P1.27mm; symbol Isolator:LTV-817S -> Tales:OR-3H4-4; Case SMDIP-4 -> SOP-16-4.4; LCSC Part # C109227 -> C2838167; Mfr Lite-On -> Orient; Mfr PN LTV-817S-TA1-C -> OR-3H4-4GB-TA1-GK; Vendor PN C109227 -> C2838167
- U12: renamed from U18; value LTV-817S -> OR-3H4-4; footprint Tales:SMDIP-4_W9.53mm -> Package_SO:SOP-16_4.4x10.4mm_P1.27mm; symbol Isolator:LTV-817S -> Tales:OR-3H4-4; Case SMDIP-4 -> SOP-16-4.4; LCSC Part # C109227 -> C2838167; Mfr Lite-On -> Orient; Mfr PN LTV-817S-TA1-C -> OR-3H4-4GB-TA1-GK; Vendor PN C109227 -> C2838167
- U12: renamed from U19; value LTV-817S -> OR-3H4-4; footprint Tales:SMDIP-4_W9.53mm -> Package_SO:SOP-16_4.4x10.4mm_P1.27mm; symbol Isolator:LTV-817S -> Tales:OR-3H4-4; Case SMDIP-4 -> SOP-16-4.4; LCSC Part # C109227 -> C2838167; Mfr Lite-On -> Orient; Mfr PN LTV-817S-TA1-C -> OR-3H4-4GB-TA1-GK; Vendor PN C109227 -> C2838167
- U12: renamed from U20; value LTV-817S -> OR-3H4-4; footprint Tales:SMDIP-4_W9.53mm -> Package_SO:SOP-16_4.4x10.4mm_P1.27mm; symbol Isolator:LTV-817S -> Tales:OR-3H4-4; Case SMDIP-4 -> SOP-16-4.4; LCSC Part # C109227 -> C2838167; Mfr Lite-On -> Orient; Mfr PN LTV-817S-TA1-C -> OR-3H4-4GB-TA1-GK; Vendor PN C109227 -> C2838167
- U12: renamed from U21; value LTV-817S -> OR-3H4-4; footprint Tales:SMDIP-4_W9.53mm -> Package_SO:SOP-16_4.4x10.4mm_P1.27mm; symbol Isolator:LTV-817S -> Tales:OR-3H4-4; Case SMDIP-4 -> SOP-16-4.4; LCSC Part # C109227 -> C2838167; Mfr Lite-On -> Orient; Mfr PN LTV-817S-TA1-C -> OR-3H4-4GB-TA1-GK; Vendor PN C109227 -> C2838167
- U13: renamed from U23; value LTV-817S -> OR-3H4-4; footprint Tales:SMDIP-4_W9.53mm -> Package_SO:SOP-16_4.4x10.4mm_P1.27mm; symbol Isolator:LTV-817S -> Tales:OR-3H4-4; Case SMDIP-4 -> SOP-16-4.4; LCSC Part # C109227 -> C2838167; Mfr Lite-On -> Orient; Mfr PN LTV-817S-TA1-C -> OR-3H4-4GB-TA1-GK; Vendor PN C109227 -> C2838167
- U13: renamed from U24; value LTV-817S -> OR-3H4-4; footprint Tales:SMDIP-4_W9.53mm -> Package_SO:SOP-16_4.4x10.4mm_P1.27mm; symbol Isolator:LTV-817S -> Tales:OR-3H4-4; Case SMDIP-4 -> SOP-16-4.4; LCSC Part # C109227 -> C2838167; Mfr Lite-On -> Orient; Mfr PN LTV-817S-TA1-C -> OR-3H4-4GB-TA1-GK; Vendor PN C109227 -> C2838167
- U13: renamed from U22; value LTV-817S -> OR-3H4-4; footprint Tales:SMDIP-4_W9.53mm -> Package_SO:SOP-16_4.4x10.4mm_P1.27mm; symbol Isolator:LTV-817S -> Tales:OR-3H4-4; Case SMDIP-4 -> SOP-16-4.4; LCSC Part # C109227 -> C2838167; Mfr Lite-On -> Orient; Mfr PN LTV-817S-TA1-C -> OR-3H4-4GB-TA1-GK; Vendor PN C109227 -> C2838167
- U13: renamed from U25; value LTV-817S -> OR-3H4-4; footprint Tales:SMDIP-4_W9.53mm -> Package_SO:SOP-16_4.4x10.4mm_P1.27mm; symbol Isolator:LTV-817S -> Tales:OR-3H4-4; Case SMDIP-4 -> SOP-16-4.4; LCSC Part # C109227 -> C2838167; Mfr Lite-On -> Orient; Mfr PN LTV-817S-TA1-C -> OR-3H4-4GB-TA1-GK; Vendor PN C109227 -> C2838167
Connections:
- net GND: now also U10.11, U10.13, U10.15, U10.4, U10.6, U10.8, U10.9, U11.11, U11.13, U11.15, U11.4, U11.6, U11.8, U11.9, U12.11, U12.13, U12.15, U12.4, U12.6, U12.8, U12.9, U13.11, U13.13, U13.15, U13.4, U13.6, U13.8, U13.9; no longer U10.2, U10.2, U10.2, U10.3, U10.3, U10.3, U10.3, U11.2, U11.2, U11.2, U11.3, U11.3, U11.3, U11.3, U12.2, U12.2, U12.2, U12.3, U12.3, U12.3, U12.3, U13.2, U13.2, U13.2, U13.3, U13.3, U13.3, U13.3
- net IN1: now also U10.16; no longer U10.4
- net IN10: now also U12.14; no longer U12.4
- net IN11: now also U12.12; no longer U12.4
- net IN12: now also U12.10; no longer U12.4
- net IN13: now also U13.16; no longer U13.4
- net IN14: now also U13.14; no longer U13.4
- net IN15: now also U13.12; no longer U13.4
- net IN16: now also U13.10; no longer U13.4
- net IN2: now also U10.14; no longer U10.4
- net IN3: now also U10.12; no longer U10.4
- net IN4: now also U10.10; no longer U10.4
- net IN5: now also U11.16; no longer U11.4
- net IN6: now also U11.14; no longer U11.4
- net IN7: now also U11.12; no longer U11.4
- net IN8: now also U11.10; no longer U11.4
- net IN9: now also U12.16; no longer U12.4
- net at D36.2 (A): now also U13.3; no longer U13.1
- net at D21.2 (A): now also U11.5; no longer U11.1
- net at D37.2 (A): now also U13.5; no longer U13.1
- net at D14.2 (A): now also U10.7; no longer U10.1
- net at D38.2 (A): now also U13.7; no longer U13.1
- net at D28.2 (A): now also U12.3; no longer U12.1
- net at D13.2 (A): now also U10.5; no longer U10.1
- net at D12.2 (A): now also U10.3; no longer U10.1
- net at D22.2 (A): now also U11.7; no longer U11.1
- net at D30.2 (A): now also U12.7; no longer U12.1
- net at D20.2 (A): now also U11.3; no longer U11.1
- net at D29.2 (A): now also U12.5; no longer U12.1

Commit message: Dev
Parts:
- D10, D15, D16, D17, D18, D23, D24, D25, D26, D31, D32, D33, D34, D7, D8, D9: value BLUE/0603 -> GREEN/0603; LCSC Part # C72041 -> C72043; Mfr PN 19-217/BHC-ZL1M2RY/3T -> 19-217/GHC-YR1S2/3T; Vendor PN C72041 -> C72043
- D11, D12, D13, D14, D19, D20, D21, D22, D27, D28, D29, D30, D35, D36, D37, D38: footprint Tales:D_MiniMELF -> Diode_SMD:D_MiniMELF; Case MiniMELF -> Mini-MELF; LCSC Part # C109072 -> C8067; Mfr PN ZMM5239B -> ZMM9V1-M; Vendor PN C109072 -> C8067
- R39, R40, R41, R42, R51, R52, R53, R54, R63, R64, R65, R66, R75, R76, R77, R78: value 1k2/0,250W/1206 -> 1k8/0,125W/0805; footprint Tales:R_1206_3216Metric -> Tales:R_0805_2012Metric; Case 1206/3216 -> 0805/2012; LCSC Part # C17891 -> C17398; Mfr PN 1206W4F1201T5E -> 0805W8F1801T5E; Vendor PN C17891 -> C17398
- R43, R44, R45, R46, R55, R56, R57, R58, R67, R68, R69, R70, R79, R80, R81, R82: value 3k3/62,5mW/0402 -> 2k2/62,5mW/0402; LCSC Part # C25890 -> C25879; Mfr PN 0402WGF3301TCE -> 0402WGF2201TCE; Vendor PN C25890 -> C25879
Other:
- note added: "ENTRADA OPTO Corrente na entrada 24V - 9,1V -1,2V = 13,7V 13,7V / 1800R = 7,62mA Potência dissipada no resistor série 1800 x SQ(0,00762) = 0,1045 104,5mW - usar resistor 125mW"
- note added: "SAÍDA OPTO CTR opto com i=8mA e Vce = 0,4V ~= 150% Corrente na saída do opto pode chegar a 12mA Corrente máxima prevista na saída do opto 3,3V - 0,4V = 2,9V 2,9V / 2200R = 1,32mA"
