File: V1/ESP-relay-32ch-V1-inputs-2.kicad_sch (KiCad schematic)
At the start: 112 parts, among them U10 LTV-817S, U11 LTV-817S, U12 LTV-817S, U13 LTV-817S, U14 LTV-817S, U15 LTV-817S, U16 LTV-817S, U17 LTV-817S, U18 LTV-817S, U3 LTV-817S, U4 LTV-817S, U5 LTV-817S, U6 LTV-817S, U7 LTV-817S, U8 LTV-817S, U9 LTV-817S

Commit message: Dev
Parts:
- U10, U11, U12, U13, U14, U15, U16, U17, U18, U3, U4, U5, U6, U7, U8, U9: value LTV-817S -> OR-3H4-4; footprint Tales:SMDIP-4_W9.53mm -> Package_SO:SOP-16_4.4x10.4mm_P1.27mm; symbol Isolator:LTV-817S -> Tales:OR-3H4-4; Case SMDIP-4 -> SOP-16-4.4; LCSC Part # C109227 -> C2838167; Mfr Lite-On -> Orient; Mfr PN LTV-817S-TA1-C -> OR-3H4-4GB-TA1-GK; Vendor PN C109227 -> C2838167
Connections:
- net GND: now also U10.15, U11.15, U12.15, U13.15, U14.15, U15.15, U16.15, U17.15, U18.15, U3.15, U4.15, U5.15, U6.15, U7.15, U8.15, U9.15; no longer U10.3, U11.3, U12.3, U13.3, U14.3, U15.3, U16.3, U17.3, U18.3, U3.3, U4.3, U5.3, U6.3, U7.3, U8.3, U9.3
- net IN17: now also U3.16; no longer U3.4
- net IN18: now also U4.16; no longer U4.4
- net IN19: now also U5.16; no longer U5.4
- net IN20: now also U6.16; no longer U6.4
- net IN21: now also U7.16; no longer U7.4
- net IN22: now also U8.16; no longer U8.4
- net IN23: now also U9.16; no longer U9.4
- net IN24: now also U10.16; no longer U10.4
- net IN25: now also U11.16; no longer U11.4
- net IN26: now also U12.16; no longer U12.4
- net IN27: now also U13.16; no longer U13.4
- net IN28: now also U14.16; no longer U14.4
- net IN29: now also U15.16; no longer U15.4
- net IN30: now also U16.16; no longer U16.4
- net IN31: now also U17.16; no longer U17.4
- net IN32: now also U18.16; no longer U18.4

Commit message: Dev
Parts:
- D10, D12, D14, D16, D18, D20, D22, D24, D26, D28, D30, D32, D34, D36, D6, D8: value BLUE/0603 -> GREEN/0603; LCSC Part # C72041 -> C72043; Mfr PN 19-217/BHC-ZL1M2RY/3T -> 19-217/GHC-YR1S2/3T; Vendor PN C72041 -> C72043
- D11, D13, D15, D17, D19, D21, D23, D25, D27, D29, D31, D33, D35, D37, D7, D9: footprint Tales:D_MiniMELF -> Diode_SMD:D_MiniMELF; Case MiniMELF -> Mini-MELF; LCSC Part # C109072 -> C8067; Mfr PN ZMM5239B -> ZMM9V1-M; Vendor PN C109072 -> C8067
- R11, R14, R17, R20, R23, R26, R29, R32, R35, R38, R41, R44, R47, R50, R53, R56: value 1k2/0,250W/1206 -> 1k8/0,125W/0805; footprint Tales:R_1206_3216Metric -> Tales:R_0805_2012Metric; Case 1206/3216 -> 0805/2012; LCSC Part # C17891 -> C17398; Mfr PN 1206W4F1201T5E -> 0805W8F1801T5E; Vendor PN C17891 -> C17398
- R12, R15, R18, R21, R24, R27, R30, R33, R36, R39, R42, R45, R48, R51, R54, R57: value 3k3/62,5mW/0402 -> 2k2/62,5mW/0402; LCSC Part # C25890 -> C25879; Mfr PN 0402WGF3301TCE -> 0402WGF2201TCE; Vendor PN C25890 -> C25879
