File: V1/ESP-relay-32ch-V1-lan.kicad_sch (KiCad schematic)
At the start: 28 parts, among them J11 ETHERNET, U5 LAN8710A

Commit message: Dev
Parts:
- R15, R18, R19, R20, R21, R22, R23, R25: value 3k3/62,5mW/0402 -> 2k2/62,5mW/0402; LCSC Part # C25890 -> C25879; Mfr PN 0402WGF3301TCE -> 0402WGF2201TCE; Vendor PN C25890 -> C25879
Changed lines of the file:
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@@
       (effects (font (size 1.27 1.27)) (justify left))
     )
-    (property "Value" "3k3/62,5mW/0402" (at 64.77 53.34 0)
+    (property "Value" "2k2/62,5mW/0402" (at 64.77 53.34 0)
       (effects (font (size 1.27 1.27)) (justify left))
     )
@@
       (effects (font (size 1.27 1.27)) hide)
     )
-    (property "Mfr PN" "0402WGF3301TCE" (at 62.23 53.34 0)
+    (property "Mfr PN" "0402WGF2201TCE" (at 62.23 53.34 0)
       (effects (font (size 1.27 1.27)) hide)
     )
@@
       (effects (font (size 1.27 1.27)) hide)
     )
-    (property "Vendor PN" "C25890" (at 62.23 53.34 0)
-      (effects (font (size 1.27 1.27)) hide)
-    )
-    (property "LCSC Part #" "C25890" (at 64.77 55.88 0)
+    (property "Vendor PN" "C25879" (at 62.23 53.34 0)
+      (effects (font (size 1.27 1.27)) hide)
+    )
+    (property "LCSC Part #" "C25879" (at 64.77 55.88 0)
       (effects (font (size 1.27 1.27)) (justify left))
     )
@@
       (effects (font (size 1.27 1.27)) (justify left))
     )
-    (property "Value" "3k3/62,5mW/0402" (at 138.43 53.34 0)
+    (property "Value" "2k2/62,5mW/0402" (at 138.43 53.34 0)
       (effects (font (size 1.27 1.27)) (justify left))
     )
@@
       (effects (font (size 1.27 1.27)) hide)
     )
-    (property "Mfr PN" "0402WGF3301TCE" (at 135.89 53.34 0)
+    (property "Mfr PN" "0402WGF2201TCE" (at 135.89 53.34 0)
       (effects (font (size 1.27 1.27)) hide)
     )
@@
       (effects (font (size 1.27 1.27)) hide)
     )
-    (property "Vendor PN" "C25890" (at 135.89 53.34 0)
-      (effects (font (size 1.27 1.27)) hide)
-    )
-    (property "LCSC Part #" "C25890" (at 138.43 55.88 0)
+    (property "Vendor PN" "C25879" (at 135.89 53.34 0)
+      (effects (font (size 1.27 1.27)) hide)
+    )
+    (property "LCSC Part #" "C25879" (at 138.43 55.88 0)
       (effects (font (size 1.27 1.27)) (justify left))
     )
@@
       (effects (font (size 1.27 1.27)) (justify left))
     )
-    (property "Value" "3k3/62,5mW/0402" (at 88.9 53.34 0)
+    (property "Value" "2k2/62,5mW/0402" (at 88.9 53.34 0)
       (effects (font (size 1.27 1.27)) (justify left))
     )
@@
       (effects (font (size 1.27 1.27)) hide)
     )
-    (property "Mfr PN" "0402WGF3301TCE" (at 86.36 53.34 0)
+    (property "Mfr PN" "0402WGF2201TCE" (at 86.36 53.34 0)
       (effects (font (size 1.27 1.27)) hide)
     )
@@
       (effects (font (size 1.27 1.27)) hide)
     )
-    (property "Vendor PN" "C25890" (at 86.36 53.34 0)
-      (effects (font (size 1.27 1.27)) hide)
-    )
-    (property "LCSC Part #" "C25890" (at 88.9 55.88 0)
+    (property "Vendor PN" "C25879" (at 86.36 53.34 0)
+      (effects (font (size 1.27 1.27)) hide)
+    )
+    (property "LCSC Part #" "C25879" (at 88.9 55.88 0)
       (effects (font (size 1.27 1.27)) (justify left))
     )
@@
       (effects (font (size 1.27 1.27)) (justify left))
     )
-    (property "Value" "3k3/62,5mW/0402" (at 124.46 96.52 0)
+    (property "Value" "2k2/62,5mW/0402" (at 124.46 96.52 0)
       (effects (font (size 1.27 1.27)) (justify left))
     )
@@
       (effects (font (size 1.27 1.27)) hide)
     )
-    (property "Mfr PN" "0402WGF3301TCE" (at 121.92 96.52 0)
+    (property "Mfr PN" "0402WGF2201TCE" (at 121.92 96.52 0)
       (effects (font (size 1.27 1.27)) hide)
     )
@@
       (effects (font (size 1.27 1.27)) hide)
     )
-    (property "Vendor PN" "C25890" (at 121.92 96.52 0)
-      (effects (font (size 1.27 1.27)) hide)
-    )
-    (property "LCSC Part #" "C25890" (at 124.46 99.06 0)
+    (property "Vendor PN" "C25879" (at 121.92 96.52 0)
+      (effects (font (size 1.27 1.27)) hide)
+    )
+    (property "LCSC Part #" "C25879" (at 124.46 99.06 0)
       (effects (font (size 1.27 1.27)) (justify left))
     )
@@
       (effects (font (size 1.27 1.27)) (justify left))
     )
-    (property "Value" "3k3/62,5mW/0402" (at 107.95 116.84 0)
+    (property "Value" "2k2/62,5mW/0402" (at 107.95 116.84 0)
       (effects (font (size 1.27 1.27)) (justify left))
     )
@@
       (effects (font (size 1.27 1.27)) hide)
     )
-    (property "Mfr PN" "0402WGF3301TCE" (at 105.41 116.84 0)
+    (property "Mfr PN" "0402WGF2201TCE" (at 105.41 116.84 0)
       (effects (font (size 1.27 1.27)) hide)
     )
@@
       (effects (font (size 1.27 1.27)) hide)
     )
-    (property "Vendor PN" "C25890" (at 105.41 116.84 0)
-      (effects (font (size 1.27 1.27)) hide)
-    )
-    (property "LCSC Part #" "C25890" (at 107.95 119.38 0)
+    (property "Vendor PN" "C25879" (at 105.41 116.84 0)
+      (effects (font (size 1.27 1.27)) hide)
+    )
+    (property "LCSC Part #" "C25879" (at 107.95 119.38 0)
       (effects (font (size 1.27 1.27)) (justify left))
     )
@@
       (effects (font (size 1.27 1.27)) (justify left))
     )
-    (property "Value" "3k3/62,5mW/0402" (at 97.79 130.81 0)
+    (property "Value" "2k2/62,5mW/0402" (at 97.79 130.81 0)
       (effects (font (size 1.27 1.27)) (justify left))
     )
@@
       (effects (font (size 1.27 1.27)) hide)
     )
-    (property "Mfr PN" "0402WGF3301TCE" (at 95.25 130.81 0)
+    (property "Mfr PN" "0402WGF2201TCE" (at 95.25 130.81 0)
       (effects (font (size 1.27 1.27)) hide)
     )
@@
       (effects (font (size 1.27 1.27)) hide)
     )
-    (property "Vendor PN" "C25890" (at 95.25 130.81 0)
-      (effects (font (size 1.27 1.27)) hide)
-    )
-    (property "LCSC Part #" "C25890" (at 97.79 133.35 0)
+    (property "Vendor PN" "C25879" (at 95.25 130.81 0)
+      (effects (font (size 1.27 1.27)) hide)
+    )
+    (property "LCSC Part #" "C25879" (at 97.79 133.35 0)
       (effects (font (size 1.27 1.27)) (justify left))
     )
@@
       (effects (font (size 1.27 1.27)) (justify left))
     )
-    (property "Value" "3k3/62,5mW/0402" (at 113.03 53.34 0)
+    (property "Value" "2k2/62,5mW/0402" (at 113.03 53.34 0)
       (effects (font (size 1.27 1.27)) (justify left))
     )
@@
       (effects (font (size 1.27 1.27)) hide)
     )
-    (property "Mfr PN" "0402WGF3301TCE" (at 110.49 53.34 0)
+    (property "Mfr PN" "0402WGF2201TCE" (at 110.49 53.34 0)
       (effects (font (size 1.27 1.27)) hide)
     )
@@
       (effects (font (size 1.27 1.27)) hide)
     )
-    (property "Vendor PN" "C25890" (at 110.49 53.34 0)
-      (effects (font (size 1.27 1.27)) hide)
-    )
-    (property "LCSC Part #" "C25890" (at 113.03 55.88 0)
+    (property "Vendor PN" "C25879" (at 110.49 53.34 0)
+      (effects (font (size 1.27 1.27)) hide)
+    )
+    (property "LCSC Part #" "C25879" (at 113.03 55.88 0)
       (effects (font (size 1.27 1.27)) (justify left))
     )
@@
       (effects (font (size 1.27 1.27)) (justify left))
     )
-    (property "Value" "3k3/62,5mW/0402" (at 40.64 53.34 0)
+    (property "Value" "2k2/62,5mW/0402" (at 40.64 53.34 0)
       (effects (font (size 1.27 1.27)) (justify left))
     )
@@
       (effects (font (size 1.27 1.27)) hide)
     )
-    (property "Mfr PN" "0402WGF3301TCE" (at 38.1 53.34 0)
+    (property "Mfr PN" "0402WGF2201TCE" (at 38.1 53.34 0)
       (effects (font (size 1.27 1.27)) hide)
     )
@@
       (effects (font (size 1.27 1.27)) hide)
     )
-    (property "Vendor PN" "C25890" (at 38.1 53.34 0)
-      (effects (font (size 1.27 1.27)) hide)
-    )
-    (property "LCSC Part #" "C25890" (at 40.64 55.88 0)
-      (effects (font (size 1.27 1.27)) (justify left))
-    )
+    (property "Vendor PN" "C25879" (at 38.1 53.34 0)
+      (effects (font (size 1.27 1.27)) hide)
+    )
+    (property "LCSC Part #" "C25879" (at 40.64 55.88 0)
+      (effects (font (size 1.27 1.27)) (justify left))
+    )
