File: V1/ESP-relay-32ch-V1-outputs-1.kicad_sch (KiCad schematic)
At the start: 80 parts, among them Q10 MMBT2222A/SOT-23-3, Q11 MMBT2222A/SOT-23-3, Q12 MMBT2222A/SOT-23-3, Q13 MMBT2222A/SOT-23-3, Q14 MMBT2222A/SOT-23-3, Q15 MMBT2222A/SOT-23-3, Q16 MMBT2222A/SOT-23-3, Q17 MMBT2222A/SOT-23-3, Q18 MMBT2222A/SOT-23-3, Q19 MMBT2222A/SOT-23-3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

Commit message: Dev
Parts:
- D71, D72, D73, D74, D75, D76, D77, D78, D79, D80, D81, D82, D83, D84, D85, D86: value BLUE/0603 -> GREEN/0603; LCSC Part # C72041 -> C72043; Mfr PN 19-217/BHC-ZL1M2RY/3T -> 19-217/GHC-YR1S2/3T; Vendor PN C72041 -> C72043
