File: V1/ESP-relay-32ch-V1 - Copia.kicad_pcb (KiCad board)
At the start: 2 copper layers, 193 x 67.8 mm, 450 parts, among them J1 Conn_01x08, J10 USB, J11 ETHERNET, J2 Conn_01x08, J3 Conn_01x08, J4 Conn_01x08, J5 Conn_01x08, J6 Conn_01x08, J7 Conn_01x08, J8 Conn_01x08, J9 VIN, Q1 WPM2015-3/TR, Q10 MMBT2222A/SOT-23-3, Q11 MMBT2222A/SOT-23-3, Q12 MMBT2222A/SOT-23-3, Q13 MMBT2222A/SOT-23-3, Q14 MMBT2222A/SOT-23-3, Q15 MMBT2222A/SOT-23-3, Q16 MMBT2222A/SOT-23-3, Q17 MMBT2222A/SOT-23-3, Q18 MMBT2222A/SOT-23-3, Q19 MMBT2222A/SOT-23-3, Q2 LMUN2211LT1G, Q20 MMBT2222A/SOT-23-3, Q21 MMBT2222A/SOT-23-3, Q22 MMBT2222A/SOT-23-3, Q23 MMBT2222A/SOT-23-3, Q24 MMBT2222A/SOT-23-3, Q25 MMBT2222A/SOT-23-3, Q26 MMBT2222A/SOT-23-3, Q27 MMBT2222A/SOT-23-3, Q28 MMBT2222A/SOT-23-3, Q29 MMBT2222A/SOT-23-3, Q3 UMH3N, Q30 MMBT2222A/SOT-23-3, Q31 MMBT2222A/SOT-23-3, Q32 MMBT2222A/SOT-23-3, Q33 MMBT2222A/SOT-23-3, Q34 MMBT2222A/SOT-23-3, Q35 MMBT2222A/SOT-23-3, Q4 MMBT2222A/SOT-23-3, Q5 MMBT2222A/SOT-23-3, Q6 MMBT2222A/SOT-23-3, Q7 MMBT2222A/SOT-23-3, Q8 MMBT2222A/SOT-23-3, Q9 MMBT2222A/SOT-23-3, SW1 RESET, U1 SY8089A1AAC, U10 OR-3H4-4, U11 OR-3H4-4, U12 OR-3H4-4, U13 OR-3H4-4, U14 OR-3H4-4, U15 OR-3H4-4, U16 OR-3H4-4, U17 OR-3H4-4, U2 TX4138, U3 CH340C, U4 ESP32-WROOM-32UE-N16, U5 LAN8710A, U6 MCP23017_SS, U7 MCP23017_SS, U8 MCP23017_SS, U9 MCP23017_SS

Commit message: Dev
Parts:
- moved Q3 13.0 mm to (195.3, 99.1)
- moved F1 11.6 mm to (190.5, 129.1), turned to -90 degrees
- moved D3 6.99 mm to (190.5, 124.8), turned to 90 degrees
- moved D76 6.35 mm to (219.1, 112.9)
- moved D80 6.35 mm to (233.0, 112.9)
- moved D92 6.35 mm to (219.1, 79.9)
- moved D96 6.35 mm to (233.0, 79.9)
- moved Q13 6.35 mm to (233.0, 116.5)
- moved Q25 6.35 mm to (219.1, 83.5)
- moved Q29 6.35 mm to (233.0, 83.5)
- moved Q9 6.35 mm to (219.1, 116.5)
- moved R131 6.35 mm to (205.1, 105.5)
- moved R138 6.35 mm to (215.3, 113.2)
- moved R143 6.35 mm to (215.3, 105.5)
- moved R146 6.35 mm to (222.9, 113.2)
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Routing:
- net GND: track 1114.9 -> 1382.0 mm
- net /MCU/I2C_SDA: track 29.4 -> 142.5 mm, vias 0 -> 3
- net /MCU/I2C_SCL: track 41.4 -> 153.3 mm, vias 0 -> 3
- net /LAN/TD+: track 0.00 -> 66.5 mm, vias 0 -> 1
- net /LAN/EMAC_RX: track 0.00 -> 63.5 mm, vias 0 -> 2
- net /LAN/EMAC_MDC: track 0.00 -> 62.1 mm, vias 0 -> 2
- net /LAN/EMAC_RXD0: track 0.00 -> 60.6 mm, vias 0 -> 2
- net /LAN/TD-: track 0.00 -> 60.1 mm, vias 0 -> 1
- net /LAN/EMAC_RXD1: track 0.00 -> 58.4 mm, vias 0 -> 2
- net Net-(Q3B-C2): track 0.00 -> 57.2 mm, vias 0 -> 4
- net +5V: track 48.1 -> 105.3 mm
- net /LAN/RD+: track 0.00 -> 56.3 mm, vias 0 -> 1
- net /LAN/EMAC_MDIO: track 0.00 -> 53.5 mm
- net Net-(U3-RXD): track 0.00 -> 53.5 mm, vias 0 -> 2
- net Net-(U3-TXD): track 0.00 -> 49.7 mm, vias 0 -> 2
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