File: V1/ESP-relay-32ch-V1-mcu.kicad_sch (KiCad schematic)
At the start: 12 parts, among them Q3 UMH3N, SW1 RESET, U3 CH340C, U4 ESP32-WROOM-32E-8MB

Commit message: Dev
Parts:
- R13, R14: value 3k3/62,5mW/0402 -> 2k2/62,5mW/0402; LCSC Part # C25890 -> C25879; Mfr PN 0402WGF3301TCE -> 0402WGF2201TCE; Vendor PN C25890 -> C25879
- U4: value ESP32-WROOM-32E-8MB -> ESP32-WROOM-32UE-N16; footprint Tales:ESP32-WROOM-32 -> Tales:ESP32-WROOM-32U; symbol RF_Module:ESP32-WROOM-32 -> RF_Module:ESP32-WROOM-32U; Case ESP32-WROOM -> ESP32-WROOM-U; LCSC Part # C701342 -> C701346; Mfr PN ESP32-WROOM-32E(8MB) -> ESP32-WROOM-32UE-N16; Vendor PN C701342 -> C701346
Changed lines of the file:
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@@
       (effects (font (size 1.27 1.27)) (justify left))
     )
-    (property "Value" "3k3/62,5mW/0402" (at 252.73 123.19 0)
+    (property "Value" "2k2/62,5mW/0402" (at 252.73 123.19 0)
       (effects (font (size 1.27 1.27)) (justify left))
     )
@@
       (effects (font (size 1.27 1.27)) hide)
     )
-    (property "Mfr PN" "0402WGF3301TCE" (at 250.19 123.19 0)
+    (property "Mfr PN" "0402WGF2201TCE" (at 250.19 123.19 0)
       (effects (font (size 1.27 1.27)) hide)
     )
@@
       (effects (font (size 1.27 1.27)) hide)
     )
-    (property "Vendor PN" "C25890" (at 250.19 123.19 0)
-      (effects (font (size 1.27 1.27)) hide)
-    )
-    (property "LCSC Part #" "C25890" (at 252.73 125.73 0)
+    (property "Vendor PN" "C25879" (at 250.19 123.19 0)
+      (effects (font (size 1.27 1.27)) hide)
+    )
+    (property "LCSC Part #" "C25879" (at 252.73 125.73 0)
       (effects (font (size 1.27 1.27)) (justify left))
     )
@@
       (effects (font (size 1.27 1.27)) (justify left))
     )
-    (property "Value" "3k3/62,5mW/0402" (at 227.33 123.19 0)
+    (property "Value" "2k2/62,5mW/0402" (at 227.33 123.19 0)
       (effects (font (size 1.27 1.27)) (justify left))
     )
@@
       (effects (font (size 1.27 1.27)) hide)
     )
-    (property "Mfr PN" "0402WGF3301TCE" (at 224.79 123.19 0)
+    (property "Mfr PN" "0402WGF2201TCE" (at 224.79 123.19 0)
       (effects (font (size 1.27 1.27)) hide)
     )
@@
       (effects (font (size 1.27 1.27)) hide)
     )
-    (property "Vendor PN" "C25890" (at 224.79 123.19 0)
-      (effects (font (size 1.27 1.27)) hide)
-    )
-    (property "LCSC Part #" "C25890" (at 227.33 125.73 0)
+    (property "Vendor PN" "C25879" (at 224.79 123.19 0)
+      (effects (font (size 1.27 1.27)) hide)
+    )
+    (property "LCSC Part #" "C25879" (at 227.33 125.73 0)
       (effects (font (size 1.27 1.27)) (justify left))
     )
@@
     )
   )
-  (symbol (lib_id "RF_Module:ESP32-WROOM-32") (at 179.07 110.49 0) (unit 1)
+  (symbol (lib_id "RF_Module:ESP32-WROOM-32U") (at 179.07 110.49 0) (unit 1)
     (in_bom yes) (on_board yes) (dnp no)
     (property "Reference" "U4" (at 182.88 146.05 0)
       (effects (font (size 1.27 1.27)) (justify left))
     )
-    (property "Value" "ESP32-WROOM-32E-8MB" (at 182.88 148.59 0)
-      (effects (font (size 1.27 1.27)) (justify left))
-    )
-    (property "Footprint" "Tales:ESP32-WROOM-32" (at 179.07 148.59 0)
-      (effects (font (size 1.27 1.27)) hide)
-    )
-    (property "Datasheet" "https://www.espressif.com/sites/default/files/documentation/esp32-wroom-32_datasheet_en.pdf" (at 171.45 109.22 0)
+    (property "Value" "ESP32-WROOM-32UE-N16" (at 182.88 148.59 0)
+      (effects (font (size 1.27 1.27)) (justify left))
+    )
+    (property "Footprint" "Tales:ESP32-WROOM-32U" (at 179.07 148.59 0)
+      (effects (font (size 1.27 1.27)) hide)
+    )
+    (property "Datasheet" "https://www.espressif.com/sites/default/files/documentation/esp32-wroom-32d_esp32-wroom-32u_datasheet_en.pdf" (at 171.45 109.22 0)
       (effects (font (size 1.27 1.27)) hide)
     )
@@
       (effects (font (size 1.27 1.27)) hide)
     )
-    (property "LCSC Part #" "C701342" (at 182.88 151.13 0)
+    (property "LCSC Part #" "C701346" (at 182.88 151.13 0)
       (effects (font (size 1.27 1.27)) (justify left))
     )
@@
       (effects (font (size 1.27 1.27)) hide)
     )
-    (property "Mfr PN" "ESP32-WROOM-32E(8MB)" (at 179.07 110.49 0)
+    (property "Mfr PN" "ESP32-WROOM-32UE-N16" (at 179.07 110.49 0)
       (effects (font (size 1.27 1.27)) hide)
     )
@@
       (effects (font (size 1.27 1.27)) hide)
     )
-    (property "Vendor PN" "C701342" (at 179.07 110.49 0)
-      (effects (font (size 1.27 1.27)) hide)
-    )
-    (property "Case" "ESP32-WROOM" (at 179.07 110.49 0)
-      (effects (font (size 1.27 1.27)) hide)
-    )
+    (property "Vendor PN" "C701346" (at 179.07 110.49 0)
+      (effects (font (size 1.27 1.27)) hide)
+    )
+    (property "Case" "ESP32-WROOM-U" (at 179.07 110.49 0)
+      (effects (font (size 1.27 1.27)) hide)
+    )

Commit message: Dev
Parts:
- SW1: footprint Tales:SW_SPST_Yuandi_TS1092SB3D2G -> Button_Switch_SMD:SW_SPST_TL3342; LCSC Part # C520860 -> C318884; Mfr Yuandi -> XKB Connectivity; Mfr PN TS-1092S-B3D2-G -> TS-1187A-B-A-B; Vendor PN C520860 -> C318884
Changed lines of the file:
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@@
       (effects (font (size 1.27 1.27)) (justify right))
     )
-    (property "Footprint" "Tales:SW_SPST_Yuandi_TS1092SB3D2G" (at 120.65 111.76 0)
+    (property "Footprint" "Button_Switch_SMD:SW_SPST_TL3342" (at 120.65 111.76 0)
       (effects (font (size 1.27 1.27)) hide)
     )
@@
       (effects (font (size 1.27 1.27)) hide)
     )
-    (property "LCSC Part #" "C520860" (at 127 114.3001 90)
+    (property "LCSC Part #" "C318884" (at 127 114.3001 90)
       (effects (font (size 1.27 1.27)) (justify right))
     )
-    (property "Mfr" "Yuandi" (at 125.73 111.76 0)
+    (property "Mfr" "XKB Connectivity" (at 125.73 111.76 0)
       (effects (font (size 1.27 1.27)) hide)
     )
-    (property "Mfr PN" "TS-1092S-B3D2-G" (at 125.73 111.76 0)
+    (property "Mfr PN" "TS-1187A-B-A-B" (at 125.73 111.76 0)
       (effects (font (size 1.27 1.27)) hide)
     )
@@
       (effects (font (size 1.27 1.27)) hide)
     )
-    (property "Vendor PN" "C520860" (at 125.73 111.76 0)
+    (property "Vendor PN" "C318884" (at 125.73 111.76 0)
       (effects (font (size 1.27 1.27)) hide)
     )
