File: V1/ESP-relay-32ch-V1-power.kicad_sch (KiCad schematic)
At the start: 34 parts, among them J10 USB, J9 VIN, Q1 WPM2015-3/TR, Q2 LMUN2211LT1G, U1 SY8089A1AAC, U2 TX4138

Commit message: Design in course.
Parts:
- J9: footprint Tales:TerminalBlock_Phoenix_PT-1,5-2-3.5-H_1x02_P3.50mm_Horizontal -> Tales:TerminalBlock_Phoenix_MKDS-3-2-5.08_1x02_P5.08mm_Horizontal
Changed lines of the file:
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@@
       (effects (font (size 1.27 1.27)))
     )
-    (property "Footprint" "Tales:TerminalBlock_Phoenix_PT-1,5-2-3.5-H_1x02_P3.50mm_Horizontal" (at 34.29 36.83 0)
+    (property "Footprint" "Tales:TerminalBlock_Phoenix_MKDS-3-2-5.08_1x02_P5.08mm_Horizontal" (at 34.29 36.83 0)
       (effects (font (size 1.27 1.27)) hide)
     )

Commit message: Dev
Parts:
- D2: value BLUE/0603 -> GREEN/0603; LCSC Part # C72041 -> C72043; Mfr PN 19-217/BHC-ZL1M2RY/3T -> 19-217/GHC-YR1S2/3T; Vendor PN C72041 -> C72043
Changed lines of the file:
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@@
       (effects (font (size 1.27 1.27)) (justify right))
     )
-    (property "Value" "BLUE/0603" (at 57.15 53.34 90)
+    (property "Value" "GREEN/0603" (at 57.15 53.34 90)
       (effects (font (size 1.27 1.27)) (justify right))
     )
@@
       (effects (font (size 1.27 1.27)) hide)
     )
-    (property "Mfr PN" "19-217/BHC-ZL1M2RY/3T" (at 54.61 53.34 0)
+    (property "Mfr PN" "19-217/GHC-YR1S2/3T" (at 54.61 53.34 0)
       (effects (font (size 1.27 1.27)) hide)
     )
@@
       (effects (font (size 1.27 1.27)) hide)
     )
-    (property "Vendor PN" "C72041" (at 54.61 53.34 0)
+    (property "Vendor PN" "C72043" (at 54.61 53.34 0)
       (effects (font (size 1.27 1.27)) hide)
     )
-    (property "LCSC Part #" "C72041" (at 57.15 55.88 90)
+    (property "LCSC Part #" "C72043" (at 57.15 55.88 90)
       (effects (font (size 1.27 1.27)) (justify right))
     )

Commit message: V1 complete
Parts:
- J10: footprint Connector_USB:USB_Micro-B_Amphenol_10118194_Horizontal -> Tales:USB_Micro-B_Amphenol_10104110_Horizontal
Changed lines of the file:
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@@
       (effects (font (size 1.27 1.27)))
     )
-    (property "Footprint" "Connector_USB:USB_Micro-B_Amphenol_10118194_Horizontal" (at 41.91 92.71 0)
+    (property "Footprint" "Tales:USB_Micro-B_Amphenol_10104110_Horizontal" (at 41.91 92.71 0)
       (effects (font (size 1.27 1.27)) hide)
     )
