File: V1/ESP-relay-32ch-V1.kicad_pcb (KiCad board)
At the start: 2 copper layers, 193 x 67.8 mm, 450 parts, among them J1 Conn_01x08, J10 USB, J11 ETHERNET, J2 Conn_01x08, J3 Conn_01x08, J4 Conn_01x08, J5 Conn_01x08, J6 Conn_01x08, J7 Conn_01x08, J8 Conn_01x08, J9 VIN, Q1 WPM2015-3/TR, Q10 MMBT2222A/SOT-23-3, Q11 MMBT2222A/SOT-23-3, Q12 MMBT2222A/SOT-23-3, Q13 MMBT2222A/SOT-23-3, Q14 MMBT2222A/SOT-23-3, Q15 MMBT2222A/SOT-23-3, Q16 MMBT2222A/SOT-23-3, Q17 MMBT2222A/SOT-23-3, Q18 MMBT2222A/SOT-23-3, Q19 MMBT2222A/SOT-23-3, Q2 LMUN2211LT1G, Q20 MMBT2222A/SOT-23-3, Q21 MMBT2222A/SOT-23-3, Q22 MMBT2222A/SOT-23-3, Q23 MMBT2222A/SOT-23-3, Q24 MMBT2222A/SOT-23-3, Q25 MMBT2222A/SOT-23-3, Q26 MMBT2222A/SOT-23-3, Q27 MMBT2222A/SOT-23-3, Q28 MMBT2222A/SOT-23-3, Q29 MMBT2222A/SOT-23-3, Q3 UMH3N, Q30 MMBT2222A/SOT-23-3, Q31 MMBT2222A/SOT-23-3, Q32 MMBT2222A/SOT-23-3, Q33 MMBT2222A/SOT-23-3, Q34 MMBT2222A/SOT-23-3, Q35 MMBT2222A/SOT-23-3, Q4 MMBT2222A/SOT-23-3, Q5 MMBT2222A/SOT-23-3, Q6 MMBT2222A/SOT-23-3, Q7 MMBT2222A/SOT-23-3, Q8 MMBT2222A/SOT-23-3, Q9 MMBT2222A/SOT-23-3, SW1 RESET, U1 SY8089A1AAC, U10 OR-3H4-4, U11 OR-3H4-4, U12 OR-3H4-4, U13 OR-3H4-4, U14 OR-3H4-4, U15 OR-3H4-4, U16 OR-3H4-4, U17 OR-3H4-4, U2 TX4138, U3 CH340C, U4 ESP32-WROOM-32UE-N16, U5 LAN8710A, U6 MCP23017_SS, U7 MCP23017_SS, U8 MCP23017_SS, U9 MCP23017_SS

Commit message: Dev
Parts:
- moved D6 18.1 mm to (174.9, 100.3), turned to 0 degrees
- moved R22 17.0 mm to (179.1, 88.8), turned to -90 degrees
- moved C17 16.3 mm to (174.5, 94.6), turned to 180 degrees
- moved R24 16.2 mm to (174.8, 93.3), turned to 0 degrees
- moved C20 15.6 mm to (181.6, 103.0), turned to 90 degrees
- moved R15 15.6 mm to (188.0, 88.8), turned to -90 degrees
- moved R25 15.6 mm to (180.3, 88.8), turned to -90 degrees
- moved R26 15.6 mm to (188.0, 103.0), turned to -90 degrees
- moved R28 14.7 mm to (182.9, 103.0), turned to -90 degrees
- moved R29 14.7 mm to (186.7, 103.0), turned to -90 degrees
- moved R18 14.5 mm to (186.7, 88.8), turned to -90 degrees
- moved R23 14.5 mm to (181.6, 88.8), turned to 90 degrees
- moved R27 14.3 mm to (184.2, 103.0), turned to -90 degrees
- moved R30 14.3 mm to (185.4, 103.0), turned to -90 degrees
- moved C18 13.9 mm to (182.9, 88.7), turned to 90 degrees
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Routing:
- net /LAN/LED_G_K: track 0.00 -> 38.1 mm
- net /LAN/EMAC_MDC: track 62.8 -> 33.0 mm, vias 2 -> 0
- net /LAN/RD-: track 60.9 -> 32.7 mm
- net /LAN/TD+: track 51.2 -> 27.0 mm
- net /LAN/TD-: track 50.3 -> 26.7 mm, vias 0 -> 2
- net /LAN/EMAC_RXD1: track 27.6 -> 50.9 mm
- net /LAN/EMAC_RXD0: track 27.3 -> 49.9 mm
- net +3.3VLAN: track 56.6 -> 38.5 mm, vias 3 -> 2
- net /LAN/EMAC_RX: track 27.7 -> 45.1 mm
- net /LAN/EMAC_TXEN: track 48.4 -> 32.4 mm, vias 2 -> 0
- net /LAN/LED_Y_A: track 0.00 -> 15.9 mm
- net /LAN/EMAC_MDIO: track 17.0 -> 29.8 mm, vias 0 -> 2
- net /LAN/EMAC_CLK: track 30.3 -> 43.0 mm
- net /LAN/EMAC_TXD0: track 42.4 -> 31.6 mm, vias 2 -> 0
- net /LAN/EMAC_TXD1: track 48.0 -> 37.4 mm, vias 0 -> 2
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
Commit message: V1 complete
Parts:
- J10: footprint Connector_USB:USB_Micro-B_Amphenol_10118194_Horizontal -> Tales:USB_Micro-B_Amphenol_10104110_Horizontal
Routing:
- net GND: track 1158.1 -> 1146.6 mm, vias 149 -> 150
Other:
- board text added: "32x IN 24VDC 32x OUT 24VDC"
- board text added: "ESP-24V-32CH-V1"
- board text added: "RESET"
- board text added: "SUPORTES PCI METALTEX SP7 1x pé macho 9 mm 1x pé fêmea 9 mm 3x espaçadores 45 mm 2x espaçadores 20 mm Comprimento total 193 mm Largura da placa 67,8 mm"
- board text added: "TMASCHIO 2023"
- board text removed: "SUPORTES PCI METALTEX SP7 1x pé macho 9 mm 1x pé fêmea 9 mm 3x espaçadores 45 mm 2x espaçador 20 mm Comprimento total 193 mm Largura da placa 67,8 mm"
