File: V1/ESP-24v-32ch-V1.kicad_pcb (KiCad board)
At the start: 2 copper layers, 193 x 67.8 mm, 450 parts, among them J1 Conn_01x08, J10 USB, J11 ETHERNET, J2 Conn_01x08, J3 Conn_01x08, J4 Conn_01x08, J5 Conn_01x08, J6 Conn_01x08, J7 Conn_01x08, J8 Conn_01x08, J9 VIN, Q1 WPM2015-3/TR, Q10 MMBT2222A/SOT-23-3, Q11 MMBT2222A/SOT-23-3, Q12 MMBT2222A/SOT-23-3, Q13 MMBT2222A/SOT-23-3, Q14 MMBT2222A/SOT-23-3, Q15 MMBT2222A/SOT-23-3, Q16 MMBT2222A/SOT-23-3, Q17 MMBT2222A/SOT-23-3, Q18 MMBT2222A/SOT-23-3, Q19 MMBT2222A/SOT-23-3, Q2 LMUN2211LT1G, Q20 MMBT2222A/SOT-23-3, Q21 MMBT2222A/SOT-23-3, Q22 MMBT2222A/SOT-23-3, Q23 MMBT2222A/SOT-23-3, Q24 MMBT2222A/SOT-23-3, Q25 MMBT2222A/SOT-23-3, Q26 MMBT2222A/SOT-23-3, Q27 MMBT2222A/SOT-23-3, Q28 MMBT2222A/SOT-23-3, Q29 MMBT2222A/SOT-23-3, Q3 UMH3N, Q30 MMBT2222A/SOT-23-3, Q31 MMBT2222A/SOT-23-3, Q32 MMBT2222A/SOT-23-3, Q33 MMBT2222A/SOT-23-3, Q34 MMBT2222A/SOT-23-3, Q35 MMBT2222A/SOT-23-3, Q4 MMBT2222A/SOT-23-3, Q5 MMBT2222A/SOT-23-3, Q6 MMBT2222A/SOT-23-3, Q7 MMBT2222A/SOT-23-3, Q8 MMBT2222A/SOT-23-3, Q9 MMBT2222A/SOT-23-3, SW1 RESET, U1 SY8089A1AAC, U10 OR-3H4-4, U11 OR-3H4-4, U12 OR-3H4-4, U13 OR-3H4-4, U14 OR-3H4-4, U15 OR-3H4-4, U16 OR-3H4-4, U17 OR-3H4-4, U2 TX4138, U3 CH340C, U4 ESP32-WROOM-32UE-N16, U5 LAN8710A, U6 MCP23017_SS, U7 MCP23017_SS, U8 MCP23017_SS, U9 MCP23017_SS

Commit message: Design optimization
Parts:
- J1, J2, J3, J4, J5, J6, J7, J8: value Conn_01x08 -> DB141V-2.54-8P; footprint Tales:TerminalBlock_Phoenix_FFKDSA1-V-2.54-8_1x08_P2.54mm_Vertical -> Tales:TerminalBlock_Dibo_DB141V-2.54-8P_1x08_P2.54mm_Vertical
- SW1: footprint Button_Switch_SMD:SW_SPST_TL3342 -> Tales:SW_SPST_TL3342
Routing:
- net Net-(D11-A): track 78.6 -> 79.7 mm

Commit message: Standarization
Parts:
- L1: footprint Tales:L_3x3_H1.5 -> Tales:L_3x3_h1.5
- L2: footprint Tales:L_12x12mm_H6mm -> Tales:L_12x12mm_h6mm
Other:
- board text added: "32X IN 24VDC 32X OUT 24VDC 2023 TMASCHIO"
- board text removed: "32x IN 24VDC 32x OUT 24VDC"
- board text removed: "TMASCHIO 2023"
