File: V1/ESP-24v-32ch-V1-expanders.kicad_sch (KiCad schematic)
At the start: 8 parts, among them U25 MCP23017_SS, U26 MCP23017_SS, U27 MCP23017_SS

Commit message: Dev
Parts:
- R31, R32, R33, R34: JLCPCB BOM (none) -> 1
Changed lines of the file:
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@@
+      (effects (font (size 1.27 1.27)) hide)
+    )
+    (property "JLCPCB BOM" "1" (at 213.36 97.79 0)
       (effects (font (size 1.27 1.27)) hide)
     )
@@
       (effects (font (size 1.27 1.27)) hide)
     )
+    (property "JLCPCB BOM" "1" (at 91.44 97.79 0)
+      (effects (font (size 1.27 1.27)) hide)
+    )
     (pin "1")
     (pin "2")
@@
     )
     (property "Vendor PN" "C11702" (at 30.48 97.79 0)
+      (effects (font (size 1.27 1.27)) hide)
+    )
+    (property "JLCPCB BOM" "1" (at 30.48 97.79 0)
       (effects (font (size 1.27 1.27)) hide)
     )
@@
       (effects (font (size 1.27 1.27)) hide)
     )
+    (property "JLCPCB BOM" "1" (at 152.4 97.79 0)
+      (effects (font (size 1.27 1.27)) hide)
+    )

Commit message: Connectors rotated 180deg
Parts:
- U25, U26, U27: footprint Package_SO:SSOP-28_5.3x10.2mm_P0.65mm -> Tales:SSOP-28_5.3x10.2mm_P0.65mm
Changed lines of the file:
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@@
       (effects (font (size 1.27 1.27)) (justify left))
     )
-    (property "Footprint" "Package_SO:SSOP-28_5.3x10.2mm_P0.65mm" (at 63.5 127 0)
+    (property "Footprint" "Tales:SSOP-28_5.3x10.2mm_P0.65mm" (at 63.5 127 0)
       (effects (font (size 1.27 1.27)) (justify left) hide)
     )
@@
       (effects (font (size 1.27 1.27)) (justify left))
     )
-    (property "Footprint" "Package_SO:SSOP-28_5.3x10.2mm_P0.65mm" (at 124.46 127 0)
+    (property "Footprint" "Tales:SSOP-28_5.3x10.2mm_P0.65mm" (at 124.46 127 0)
       (effects (font (size 1.27 1.27)) (justify left) hide)
     )
@@
       (effects (font (size 1.27 1.27)) (justify left))
     )
-    (property "Footprint" "Package_SO:SSOP-28_5.3x10.2mm_P0.65mm" (at 185.42 127 0)
+    (property "Footprint" "Tales:SSOP-28_5.3x10.2mm_P0.65mm" (at 185.42 127 0)
       (effects (font (size 1.27 1.27)) (justify left) hide)
     )
@@
       (effects (font (size 1.27 1.27)) (justify left))
     )
-    (property "Footprint" "Package_SO:SSOP-28_5.3x10.2mm_P0.65mm" (at 246.38 127 0)
+    (property "Footprint" "Tales:SSOP-28_5.3x10.2mm_P0.65mm" (at 246.38 127 0)
       (effects (font (size 1.27 1.27)) (justify left) hide)
     )
