File: V1/ESP-24v-32ch-V1-inputs-1.kicad_sch (KiCad schematic)
At the start: 100 parts, among them U10 OR-3H4-4, U11 OR-3H4-4, U12 OR-3H4-4, U13 OR-3H4-4

Commit message: Project rename
Other:
- title: ESP 16x 24VDC Input 16x External Relay Output Module -> ESP 32x 24VDC Input 32x 24VDC Output Module

Commit message: Connectors rotated 180deg
Parts:
- D11, D12, D13, D14, D19, D20, D21, D22, D27, D28, D29, D30, D35, D36, D37, D38: footprint Diode_SMD:D_MiniMELF -> Tales:D_MiniMELF
- U10, U11, U12, U13: footprint Package_SO:SOP-16_4.4x10.4mm_P1.27mm -> Tales:SOP-16_4.4x10.4mm_P1.27mm
Changed lines of the file:
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@@
       (effects (font (size 1.27 1.27)) (justify left))
     )
-    (property "Footprint" "Package_SO:SOP-16_4.4x10.4mm_P1.27mm" (at 247.65 78.74 0)
+    (property "Footprint" "Tales:SOP-16_4.4x10.4mm_P1.27mm" (at 247.65 78.74 0)
       (effects (font (size 1.27 1.27) italic) (justify left) hide)
     )
@@
       (effects (font (size 1.27 1.27)) (justify left))
     )
-    (property "Footprint" "Diode_SMD:D_MiniMELF" (at 111.76 107.95 90)
+    (property "Footprint" "Tales:D_MiniMELF" (at 111.76 107.95 90)
       (effects (font (size 1.27 1.27)) hide)
     )
@@
       (effects (font (size 1.27 1.27)) (justify left))
     )
-    (property "Footprint" "Package_SO:SOP-16_4.4x10.4mm_P1.27mm" (at 247.65 115.57 0)
+    (property "Footprint" "Tales:SOP-16_4.4x10.4mm_P1.27mm" (at 247.65 115.57 0)
       (effects (font (size 1.27 1.27) italic) (justify left) hide)
     )
@@
       (effects (font (size 1.27 1.27)) (justify left))
     )
-    (property "Footprint" "Diode_SMD:D_MiniMELF" (at 46.99 144.78 90)
+    (property "Footprint" "Tales:D_MiniMELF" (at 46.99 144.78 90)
       (effects (font (size 1.27 1.27)) hide)
     )
@@
       (effects (font (size 1.27 1.27)) (justify left))
     )
-    (property "Footprint" "Diode_SMD:D_MiniMELF" (at 46.99 34.29 90)
+    (property "Footprint" "Tales:D_MiniMELF" (at 46.99 34.29 90)
       (effects (font (size 1.27 1.27)) hide)
     )
@@
       (effects (font (size 1.27 1.27)) (justify left))
     )
-    (property "Footprint" "Package_SO:SOP-16_4.4x10.4mm_P1.27mm" (at 247.65 41.91 0)
+    (property "Footprint" "Tales:SOP-16_4.4x10.4mm_P1.27mm" (at 247.65 41.91 0)
       (effects (font (size 1.27 1.27) italic) (justify left) hide)
     )
@@
       (effects (font (size 1.27 1.27)) (justify left))
     )
-    (property "Footprint" "Package_SO:SOP-16_4.4x10.4mm_P1.27mm" (at 247.65 152.4 0)
+    (property "Footprint" "Tales:SOP-16_4.4x10.4mm_P1.27mm" (at 247.65 152.4 0)
       (effects (font (size 1.27 1.27) italic) (justify left) hide)
     )
@@
       (effects (font (size 1.27 1.27)) (justify left))
     )
-    (property "Footprint" "Package_SO:SOP-16_4.4x10.4mm_P1.27mm" (at 182.88 41.91 0)
+    (property "Footprint" "Tales:SOP-16_4.4x10.4mm_P1.27mm" (at 182.88 41.91 0)
       (effects (font (size 1.27 1.27) italic) (justify left) hide)
     )
@@
       (effects (font (size 1.27 1.27)) (justify left))
     )
-    (property "Footprint" "Package_SO:SOP-16_4.4x10.4mm_P1.27mm" (at 182.88 78.74 0)
+    (property "Footprint" "Tales:SOP-16_4.4x10.4mm_P1.27mm" (at 182.88 78.74 0)
       (effects (font (size 1.27 1.27) italic) (justify left) hide)
     )
@@
       (effects (font (size 1.27 1.27)) (justify left))
     )
-    (property "Footprint" "Diode_SMD:D_MiniMELF" (at 46.99 107.95 90)
+    (property "Footprint" "Tales:D_MiniMELF" (at 46.99 107.95 90)
       (effects (font (size 1.27 1.27)) hide)
     )
@@
       (effects (font (size 1.27 1.27)) (justify left))
     )
-    (property "Footprint" "Diode_SMD:D_MiniMELF" (at 241.3 34.29 90)
+    (property "Footprint" "Tales:D_MiniMELF" (at 241.3 34.29 90)
       (effects (font (size 1.27 1.27)) hide)
     )
@@
       (effects (font (size 1.27 1.27)) (justify left))
     )
-    (property "Footprint" "Diode_SMD:D_MiniMELF" (at 46.99 71.12 90)
+    (property "Footprint" "Tales:D_MiniMELF" (at 46.99 71.12 90)
       (effects (font (size 1.27 1.27)) hide)
     )
@@
       (effects (font (size 1.27 1.27)) (justify left))
     )
-    (property "Footprint" "Package_SO:SOP-16_4.4x10.4mm_P1.27mm" (at 53.34 115.57 0)
+    (property "Footprint" "Tales:SOP-16_4.4x10.4mm_P1.27mm" (at 53.34 115.57 0)
       (effects (font (size 1.27 1.27) italic) (justify left) hide)
     )
@@
       (effects (font (size 1.27 1.27)) (justify left))
     )
-    (property "Footprint" "Diode_SMD:D_MiniMELF" (at 111.76 144.78 90)
+    (property "Footprint" "Tales:D_MiniMELF" (at 111.76 144.78 90)
       (effects (font (size 1.27 1.27)) hide)
     )
@@
       (effects (font (size 1.27 1.27)) (justify left))
     )
-    (property "Footprint" "Diode_SMD:D_MiniMELF" (at 111.76 34.29 90)
+    (property "Footprint" "Tales:D_MiniMELF" (at 111.76 34.29 90)
       (effects (font (size 1.27 1.27)) hide)
     )
@@
       (effects (font (size 1.27 1.27)) (justify left))
     )
-    (property "Footprint" "Diode_SMD:D_MiniMELF" (at 176.53 144.78 90)
+    (property "Footprint" "Tales:D_MiniMELF" (at 176.53 144.78 90)
       (effects (font (size 1.27 1.27)) hide)
     )
@@
       (effects (font (size 1.27 1.27)) (justify left))
     )
-    (property "Footprint" "Package_SO:SOP-16_4.4x10.4mm_P1.27mm" (at 118.11 41.91 0)
+    (property "Footprint" "Tales:SOP-16_4.4x10.4mm_P1.27mm" (at 118.11 41.91 0)
       (effects (font (size 1.27 1.27) italic) (justify left) hide)
     )
@@
       (effects (font (size 1.27 1.27)) (justify left))
     )
-    (property "Footprint" "Diode_SMD:D_MiniMELF" (at 111.76 71.12 90)
+    (property "Footprint" "Tales:D_MiniMELF" (at 111.76 71.12 90)
       (effects (font (size 1.27 1.27)) hide)
     )
@@
       (effects (font (size 1.27 1.27)) (justify left))
     )
-    (property "Footprint" "Package_SO:SOP-16_4.4x10.4mm_P1.27mm" (at 182.88 115.57 0)
+    (property "Footprint" "Tales:SOP-16_4.4x10.4mm_P1.27mm" (at 182.88 115.57 0)
       (effects (font (size 1.27 1.27) italic) (justify left) hide)
     )
@@
       (effects (font (size 1.27 1.27)) (justify left))
     )
-    (property "Footprint" "Package_SO:SOP-16_4.4x10.4mm_P1.27mm" (at 118.11 115.57 0)
+    (property "Footprint" "Tales:SOP-16_4.4x10.4mm_P1.27mm" (at 118.11 115.57 0)
       (effects (font (size 1.27 1.27) italic) (justify left) hide)
     )
@@
       (effects (font (size 1.27 1.27)) (justify left))
     )
-    (property "Footprint" "Package_SO:SOP-16_4.4x10.4mm_P1.27mm" (at 53.34 41.91 0)
+    (property "Footprint" "Tales:SOP-16_4.4x10.4mm_P1.27mm" (at 53.34 41.91 0)
       (effects (font (size 1.27 1.27) italic) (justify left) hide)
     )
@@
       (effects (font (size 1.27 1.27)) (justify left))
     )
-    (property "Footprint" "Package_SO:SOP-16_4.4x10.4mm_P1.27mm" (at 53.34 78.74 0)
+    (property "Footprint" "Tales:SOP-16_4.4x10.4mm_P1.27mm" (at 53.34 78.74 0)
       (effects (font (size 1.27 1.27) italic) (justify left) hide)
     )
@@
       (effects (font (size 1.27 1.27)) (justify left))
     )
-    (property "Footprint" "Diode_SMD:D_MiniMELF" (at 176.53 107.95 90)
+    (property "Footprint" "Tales:D_MiniMELF" (at 176.53 107.95 90)
       (effects (font (size 1.27 1.27)) hide)
     )
@@
       (effects (font (size 1.27 1.27)) (justify left))
     )
-    (property "Footprint" "Diode_SMD:D_MiniMELF" (at 241.3 71.12 90)
+    (property "Footprint" "Tales:D_MiniMELF" (at 241.3 71.12 90)
       (effects (font (size 1.27 1.27)) hide)
     )
@@
       (effects (font (size 1.27 1.27)) (justify left))
     )
-    (property "Footprint" "Package_SO:SOP-16_4.4x10.4mm_P1.27mm" (at 53.34 152.4 0)
+    (property "Footprint" "Tales:SOP-16_4.4x10.4mm_P1.27mm" (at 53.34 152.4 0)
       (effects (font (size 1.27 1.27) italic) (justify left) hide)
     )
@@
       (effects (font (size 1.27 1.27)) (justify left))
     )
-    (property "Footprint" "Diode_SMD:D_MiniMELF" (at 241.3 107.95 90)
+    (property "Footprint" "Tales:D_MiniMELF" (at 241.3 107.95 90)
       (effects (font (size 1.27 1.27)) hide)
     )
@@
       (effects (font (size 1.27 1.27)) (justify left))
     )
-    (property "Footprint" "Package_SO:SOP-16_4.4x10.4mm_P1.27mm" (at 182.88 152.4 0)
+    (property "Footprint" "Tales:SOP-16_4.4x10.4mm_P1.27mm" (at 182.88 152.4 0)
       (effects (font (size 1.27 1.27) italic) (justify left) hide)
     )
@@
       (effects (font (size 1.27 1.27)) (justify left))
     )
-    (property "Footprint" "Package_SO:SOP-16_4.4x10.4mm_P1.27mm" (at 118.11 152.4 0)
+    (property "Footprint" "Tales:SOP-16_4.4x10.4mm_P1.27mm" (at 118.11 152.4 0)
       (effects (font (size 1.27 1.27) italic) (justify left) hide)
     )
@@
       (effects (font (size 1.27 1.27)) (justify left))
     )
-    (property "Footprint" "Package_SO:SOP-16_4.4x10.4mm_P1.27mm" (at 118.11 78.74 0)
+    (property "Footprint" "Tales:SOP-16_4.4x10.4mm_P1.27mm" (at 118.11 78.74 0)
       (effects (font (size 1.27 1.27) italic) (justify left) hide)
     )
@@
       (effects (font (size 1.27 1.27)) (justify left))
     )
-    (property "Footprint" "Diode_SMD:D_MiniMELF" (at 241.3 144.78 90)
+    (property "Footprint" "Tales:D_MiniMELF" (at 241.3 144.78 90)
       (effects (font (size 1.27 1.27)) hide)
     )
@@
       (effects (font (size 1.27 1.27)) (justify left))
     )
-    (property "Footprint" "Diode_SMD:D_MiniMELF" (at 176.53 71.12 90)
+    (property "Footprint" "Tales:D_MiniMELF" (at 176.53 71.12 90)
       (effects (font (size 1.27 1.27)) hide)
     )
@@
       (effects (font (size 1.27 1.27)) (justify left))
     )
-    (property "Footprint" "Diode_SMD:D_MiniMELF" (at 176.53 34.29 90)
+    (property "Footprint" "Tales:D_MiniMELF" (at 176.53 34.29 90)
       (effects (font (size 1.27 1.27)) hide)
     )

Commit message: Renamed to lowercase
Parts:
- renumbered C23 to C39, C24 to C40, C25 to C41, C26 to C42, C27 to C43, C28 to C44, C29 to C45, C30 to C46, C31 to C47, C32 to C48, C33 to C49, C34 to C50, C35 to C51, C36 to C52, C37 to C53, C38 to C54, D7 to D55, D8 to D56, D9 to D57, D10 to D58, D11 to D59, D12 to D60, D13 to D61, D14 to D62, D15 to D63, D16 to D64, D17 to D65, D18 to D66, D19 to D67, D20 to D68, D21 to D69, D22 to D70, D23 to D71, D24 to D72, D25 to D73, D26 to D74, D27 to D75, D28 to D76, D29 to D77, D30 to D78, D31 to D79, D32 to D80, D33 to D81, D34 to D82, D35 to D83, D36 to D84, D37 to D85, D38 to D86, R35 to R131, R36 to R132, R37 to R133, R38 to R134, R39 to R135, R40 to R136, R41 to R137, R42 to R138, R43 to R139, R44 to R140, R45 to R141, R46 to R142, R47 to R143, R48 to R144, R49 to R145, R50 to R146, R51 to R147, R52 to R148, R53 to R149, R54 to R150, R55 to R151, R56 to R152, R57 to R153, R58 to R154, R59 to R155, R60 to R156, R61 to R157, R62 to R158, R63 to R159, R64 to R160, R65 to R161, R66 to R162, R67 to R163, R68 to R164, R69 to R165, R70 to R166, R71 to R167, R72 to R168, R73 to R169, R74 to R170, R75 to R171, R76 to R172, R77 to R173, R78 to R174, R79 to R175, R80 to R176, R81 to R177, R82 to R178, U10 to U26, U10 to U27, U10 to U28, U10 to U29, U11 to U30, U11 to U31, U11 to U32, U11 to U33, U12 to U34, U12 to U35, U12 to U36, U12 to U37, U13 to U38, U13 to U39, U13 to U40, U13 to U41
Connections:
- net GND: now also U27.15, U27.2, U28.15, U28.2, U29.15, U29.2, U31.15, U31.2, U32.15, U32.2, U33.15, U33.2, U35.15, U35.2, U36.15, U36.2, U37.15, U37.2, U39.15, U39.2, U40.15, U40.2, U41.15, U41.2; no longer U27.13, U27.4, U28.11, U28.6, U29.8, U29.9, U31.13, U31.4, U32.11, U32.6, U33.8, U33.9, U35.13, U35.4, U36.11, U36.6, U37.8, U37.9, U39.13, U39.4, U40.11, U40.6, U41.8, U41.9
- net IN10: now also U35.16; no longer U35.14
- net IN11: now also U36.16; no longer U36.12
- net IN12: now also U37.16; no longer U37.10
- net IN14: now also U39.16; no longer U39.14
- net IN15: now also U40.16; no longer U40.12
- net IN16: now also U41.16; no longer U41.10
- net IN2: now also U27.16; no longer U27.14
- net IN3: now also U28.16; no longer U28.12
- net IN4: now also U29.16; no longer U29.10
- net IN6: now also U31.16; no longer U31.14
- net IN7: now also U32.16; no longer U32.12
- net IN8: now also U33.16; no longer U33.10
- net at D84.2 (A): now also U39.1; no longer U39.3
- net at D69.2 (A): now also U32.1; no longer U32.5
- net at D85.2 (A): now also U40.1; no longer U40.5
- net at D62.2 (A): now also U29.1; no longer U29.7
- net at D86.2 (A): now also U41.1; no longer U41.7
- net at D76.2 (A): now also U35.1; no longer U35.3
- net at D61.2 (A): now also U28.1; no longer U28.5
- net at D60.2 (A): now also U27.1; no longer U27.3
- net at D70.2 (A): now also U33.1; no longer U33.7
- net at D78.2 (A): now also U37.1; no longer U37.7
- net at D68.2 (A): now also U31.1; no longer U31.3
- net at D77.2 (A): now also U36.1; no longer U36.5
