File: V1/ESP-24v-32ch-V1-inputs-2.kicad_sch (KiCad schematic)
At the start: 112 parts, among them U10 OR-3H4-4, U11 OR-3H4-4, U12 OR-3H4-4, U13 OR-3H4-4, U14 OR-3H4-4, U15 OR-3H4-4, U16 OR-3H4-4, U17 OR-3H4-4, U18 OR-3H4-4, U3 OR-3H4-4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

Commit message: Project rename
Other:
- title: ESP 16x 24VDC Input 16x External Relay Output Module -> ESP 32x 24VDC Input 32x 24VDC Output Module

Commit message: Connectors rotated 180deg
Parts:
- D11, D13, D15, D17, D19, D21, D23, D25, D27, D29, D31, D33, D35, D37, D7, D9: footprint Diode_SMD:D_MiniMELF -> Tales:D_MiniMELF
- U10, U11, U12, U13, U14, U15, U16, U17, U18, U3, U4, U5, U6, U7, U8, U9: footprint Package_SO:SOP-16_4.4x10.4mm_P1.27mm -> Tales:SOP-16_4.4x10.4mm_P1.27mm
Changed lines of the file:
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@@
       (effects (font (size 1.27 1.27)) (justify left))
     )
-    (property "Footprint" "Package_SO:SOP-16_4.4x10.4mm_P1.27mm" (at 182.88 41.91 0)
+    (property "Footprint" "Tales:SOP-16_4.4x10.4mm_P1.27mm" (at 182.88 41.91 0)
       (effects (font (size 1.27 1.27) italic) (justify left) hide)
     )
@@
       (effects (font (size 1.27 1.27)) (justify left))
     )
-    (property "Footprint" "Diode_SMD:D_MiniMELF" (at 46.99 34.29 90)
+    (property "Footprint" "Tales:D_MiniMELF" (at 46.99 34.29 90)
       (effects (font (size 1.27 1.27)) hide)
     )
@@
       (effects (font (size 1.27 1.27)) (justify left))
     )
-    (property "Footprint" "Diode_SMD:D_MiniMELF" (at 241.3 34.29 90)
+    (property "Footprint" "Tales:D_MiniMELF" (at 241.3 34.29 90)
       (effects (font (size 1.27 1.27)) hide)
     )
@@
       (effects (font (size 1.27 1.27)) (justify left))
     )
-    (property "Footprint" "Diode_SMD:D_MiniMELF" (at 111.76 144.78 90)
+    (property "Footprint" "Tales:D_MiniMELF" (at 111.76 144.78 90)
       (effects (font (size 1.27 1.27)) hide)
     )
@@
       (effects (font (size 1.27 1.27)) (justify left))
     )
-    (property "Footprint" "Diode_SMD:D_MiniMELF" (at 111.76 34.29 90)
+    (property "Footprint" "Tales:D_MiniMELF" (at 111.76 34.29 90)
       (effects (font (size 1.27 1.27)) hide)
     )
@@
       (effects (font (size 1.27 1.27)) (justify left))
     )
-    (property "Footprint" "Package_SO:SOP-16_4.4x10.4mm_P1.27mm" (at 118.11 78.74 0)
+    (property "Footprint" "Tales:SOP-16_4.4x10.4mm_P1.27mm" (at 118.11 78.74 0)
       (effects (font (size 1.27 1.27) italic) (justify left) hide)
     )
@@
       (effects (font (size 1.27 1.27)) (justify left))
     )
-    (property "Footprint" "Package_SO:SOP-16_4.4x10.4mm_P1.27mm" (at 53.34 41.91 0)
+    (property "Footprint" "Tales:SOP-16_4.4x10.4mm_P1.27mm" (at 53.34 41.91 0)
       (effects (font (size 1.27 1.27) italic) (justify left) hide)
     )
@@
       (effects (font (size 1.27 1.27)) (justify left))
     )
-    (property "Footprint" "Diode_SMD:D_MiniMELF" (at 111.76 107.95 90)
+    (property "Footprint" "Tales:D_MiniMELF" (at 111.76 107.95 90)
       (effects (font (size 1.27 1.27)) hide)
     )
@@
       (effects (font (size 1.27 1.27)) (justify left))
     )
-    (property "Footprint" "Package_SO:SOP-16_4.4x10.4mm_P1.27mm" (at 53.34 78.74 0)
+    (property "Footprint" "Tales:SOP-16_4.4x10.4mm_P1.27mm" (at 53.34 78.74 0)
       (effects (font (size 1.27 1.27) italic) (justify left) hide)
     )
@@
       (effects (font (size 1.27 1.27)) (justify left))
     )
-    (property "Footprint" "Package_SO:SOP-16_4.4x10.4mm_P1.27mm" (at 247.65 41.91 0)
+    (property "Footprint" "Tales:SOP-16_4.4x10.4mm_P1.27mm" (at 247.65 41.91 0)
       (effects (font (size 1.27 1.27) italic) (justify left) hide)
     )
@@
       (effects (font (size 1.27 1.27)) (justify left))
     )
-    (property "Footprint" "Diode_SMD:D_MiniMELF" (at 111.76 71.12 90)
+    (property "Footprint" "Tales:D_MiniMELF" (at 111.76 71.12 90)
       (effects (font (size 1.27 1.27)) hide)
     )
@@
       (effects (font (size 1.27 1.27)) (justify left))
     )
-    (property "Footprint" "Diode_SMD:D_MiniMELF" (at 241.3 71.12 90)
+    (property "Footprint" "Tales:D_MiniMELF" (at 241.3 71.12 90)
       (effects (font (size 1.27 1.27)) hide)
     )
@@
       (effects (font (size 1.27 1.27)) (justify left))
     )
-    (property "Footprint" "Diode_SMD:D_MiniMELF" (at 241.3 144.78 90)
+    (property "Footprint" "Tales:D_MiniMELF" (at 241.3 144.78 90)
       (effects (font (size 1.27 1.27)) hide)
     )
@@
       (effects (font (size 1.27 1.27)) (justify left))
     )
-    (property "Footprint" "Diode_SMD:D_MiniMELF" (at 176.53 107.95 90)
+    (property "Footprint" "Tales:D_MiniMELF" (at 176.53 107.95 90)
       (effects (font (size 1.27 1.27)) hide)
     )
@@
       (effects (font (size 1.27 1.27)) (justify left))
     )
-    (property "Footprint" "Diode_SMD:D_MiniMELF" (at 46.99 107.95 90)
+    (property "Footprint" "Tales:D_MiniMELF" (at 46.99 107.95 90)
       (effects (font (size 1.27 1.27)) hide)
     )
@@
       (effects (font (size 1.27 1.27)) (justify left))
     )
-    (property "Footprint" "Package_SO:SOP-16_4.4x10.4mm_P1.27mm" (at 118.11 115.57 0)
+    (property "Footprint" "Tales:SOP-16_4.4x10.4mm_P1.27mm" (at 118.11 115.57 0)
       (effects (font (size 1.27 1.27) italic) (justify left) hide)
     )
@@
       (effects (font (size 1.27 1.27)) (justify left))
     )
-    (property "Footprint" "Diode_SMD:D_MiniMELF" (at 176.53 71.12 90)
+    (property "Footprint" "Tales:D_MiniMELF" (at 176.53 71.12 90)
       (effects (font (size 1.27 1.27)) hide)
     )
@@
       (effects (font (size 1.27 1.27)) (justify left))
     )
-    (property "Footprint" "Package_SO:SOP-16_4.4x10.4mm_P1.27mm" (at 247.65 152.4 0)
+    (property "Footprint" "Tales:SOP-16_4.4x10.4mm_P1.27mm" (at 247.65 152.4 0)
       (effects (font (size 1.27 1.27) italic) (justify left) hide)
     )
@@
       (effects (font (size 1.27 1.27)) (justify left))
     )
-    (property "Footprint" "Package_SO:SOP-16_4.4x10.4mm_P1.27mm" (at 247.65 115.57 0)
+    (property "Footprint" "Tales:SOP-16_4.4x10.4mm_P1.27mm" (at 247.65 115.57 0)
       (effects (font (size 1.27 1.27) italic) (justify left) hide)
     )
@@
       (effects (font (size 1.27 1.27)) (justify left))
     )
-    (property "Footprint" "Diode_SMD:D_MiniMELF" (at 241.3 107.95 90)
+    (property "Footprint" "Tales:D_MiniMELF" (at 241.3 107.95 90)
       (effects (font (size 1.27 1.27)) hide)
     )
@@
       (effects (font (size 1.27 1.27)) (justify left))
     )
-    (property "Footprint" "Package_SO:SOP-16_4.4x10.4mm_P1.27mm" (at 53.34 152.4 0)
+    (property "Footprint" "Tales:SOP-16_4.4x10.4mm_P1.27mm" (at 53.34 152.4 0)
       (effects (font (size 1.27 1.27) italic) (justify left) hide)
     )
@@
       (effects (font (size 1.27 1.27)) (justify left))
     )
-    (property "Footprint" "Package_SO:SOP-16_4.4x10.4mm_P1.27mm" (at 182.88 152.4 0)
+    (property "Footprint" "Tales:SOP-16_4.4x10.4mm_P1.27mm" (at 182.88 152.4 0)
       (effects (font (size 1.27 1.27) italic) (justify left) hide)
     )
@@
       (effects (font (size 1.27 1.27)) (justify left))
     )
-    (property "Footprint" "Diode_SMD:D_MiniMELF" (at 46.99 144.78 90)
+    (property "Footprint" "Tales:D_MiniMELF" (at 46.99 144.78 90)
       (effects (font (size 1.27 1.27)) hide)
     )
@@
       (effects (font (size 1.27 1.27)) (justify left))
     )
-    (property "Footprint" "Diode_SMD:D_MiniMELF" (at 46.99 71.12 90)
+    (property "Footprint" "Tales:D_MiniMELF" (at 46.99 71.12 90)
       (effects (font (size 1.27 1.27)) hide)
     )
@@
       (effects (font (size 1.27 1.27)) (justify left))
     )
-    (property "Footprint" "Package_SO:SOP-16_4.4x10.4mm_P1.27mm" (at 182.88 78.74 0)
+    (property "Footprint" "Tales:SOP-16_4.4x10.4mm_P1.27mm" (at 182.88 78.74 0)
       (effects (font (size 1.27 1.27) italic) (justify left) hide)
     )
@@
       (effects (font (size 1.27 1.27)) (justify left))
     )
-    (property "Footprint" "Package_SO:SOP-16_4.4x10.4mm_P1.27mm" (at 118.11 152.4 0)
+    (property "Footprint" "Tales:SOP-16_4.4x10.4mm_P1.27mm" (at 118.11 152.4 0)
       (effects (font (size 1.27 1.27) italic) (justify left) hide)
     )
@@
       (effects (font (size 1.27 1.27)) (justify left))
     )
-    (property "Footprint" "Diode_SMD:D_MiniMELF" (at 176.53 144.78 90)
+    (property "Footprint" "Tales:D_MiniMELF" (at 176.53 144.78 90)
       (effects (font (size 1.27 1.27)) hide)
     )
@@
       (effects (font (size 1.27 1.27)) (justify left))
     )
-    (property "Footprint" "Diode_SMD:D_MiniMELF" (at 176.53 34.29 90)
+    (property "Footprint" "Tales:D_MiniMELF" (at 176.53 34.29 90)
       (effects (font (size 1.27 1.27)) hide)
     )
@@
       (effects (font (size 1.27 1.27)) (justify left))
     )
-    (property "Footprint" "Package_SO:SOP-16_4.4x10.4mm_P1.27mm" (at 53.34 115.57 0)
+    (property "Footprint" "Tales:SOP-16_4.4x10.4mm_P1.27mm" (at 53.34 115.57 0)
       (effects (font (size 1.27 1.27) italic) (justify left) hide)
     )
@@
       (effects (font (size 1.27 1.27)) (justify left))
     )
-    (property "Footprint" "Package_SO:SOP-16_4.4x10.4mm_P1.27mm" (at 118.11 41.91 0)
+    (property "Footprint" "Tales:SOP-16_4.4x10.4mm_P1.27mm" (at 118.11 41.91 0)
       (effects (font (size 1.27 1.27) italic) (justify left) hide)
     )
@@
       (effects (font (size 1.27 1.27)) (justify left))
     )
-    (property "Footprint" "Package_SO:SOP-16_4.4x10.4mm_P1.27mm" (at 247.65 78.74 0)
+    (property "Footprint" "Tales:SOP-16_4.4x10.4mm_P1.27mm" (at 247.65 78.74 0)
       (effects (font (size 1.27 1.27) italic) (justify left) hide)
     )
@@
       (effects (font (size 1.27 1.27)) (justify left))
     )
-    (property "Footprint" "Package_SO:SOP-16_4.4x10.4mm_P1.27mm" (at 182.88 115.57 0)
+    (property "Footprint" "Tales:SOP-16_4.4x10.4mm_P1.27mm" (at 182.88 115.57 0)
       (effects (font (size 1.27 1.27) italic) (justify left) hide)
     )
