File: V1/ESP-24v-32ch-V1-lan.kicad_sch (KiCad schematic)
At the start: 28 parts, among them J11 ETHERNET, U5 LAN8710A

Commit message: Project rename
Other:
- title: ESP 16x 24VDC Input 16x External Relay Output Module -> ESP 32x 24VDC Input 32x 24VDC Output Module

Commit message: Dev
Parts:
- C15, C18, C19, C20: value 0,1uF/16V/0402 -> 0,1uF/50V/0402; LCSC Part # C1525 -> C307331; Mfr PN CL05B104KO5NNNC -> CL05B104KB54PNC; Vendor PN C1525 -> C307331
- C16, C17: value 10uF/6,3V/0603 -> 10uF/10V/0603; LCSC Part # C1691 -> C19702; Mfr PN CL10A106MQ8NNNC -> CL10A106KP8NNNC; Vendor PN C1691 -> C19702
- C21: value 1uF/6,3V/0402 -> 1uF/25V/0402; LCSC Part # C107372 -> C52923; Mfr PN CL05A105KQ5NNNC -> CL05A105KA5NQNC; Vendor PN C107372 -> C52923
- C22: value 470pF/16V/0402 -> 470pF/50V/0402; LCSC Part # C541379 -> C1537; Mfr Yageo -> FH; Mfr PN CC0402KRX7R7BB471 -> 0402B471K500NT; Vendor PN C541379 -> C1537
- R24: LCSC Part # C25890 -> C25744; Vendor PN C25890 -> C25744
Changed lines of the file:
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@@
       (effects (font (size 1.27 1.27)) (justify left))
     )
-    (property "Value" "0,1uF/16V/0402" (at 209.55 43.18 0)
+    (property "Value" "0,1uF/50V/0402" (at 209.55 43.18 0)
       (effects (font (size 1.27 1.27)) (justify left))
     )
@@
       (effects (font (size 1.27 1.27)) hide)
     )
-    (property "LCSC Part #" "C1525" (at 209.55 48.2538 0)
+    (property "LCSC Part #" "C307331" (at 209.55 48.2538 0)
       (effects (font (size 1.27 1.27)) (justify left))
     )
@@
       (effects (font (size 1.27 1.27)) hide)
     )
-    (property "Mfr PN" "CL05B104KO5NNNC" (at 207.01 43.18 0)
+    (property "Mfr PN" "CL05B104KB54PNC" (at 207.01 43.18 0)
       (effects (font (size 1.27 1.27)) hide)
     )
@@
       (effects (font (size 1.27 1.27)) hide)
     )
-    (property "Vendor PN" "C1525" (at 207.01 43.18 0)
+    (property "Vendor PN" "C307331" (at 207.01 43.18 0)
       (effects (font (size 1.27 1.27)) hide)
     )
@@
       (effects (font (size 1.27 1.27)) hide)
     )
-    (property "Vendor PN" "C25890" (at 130.81 121.92 0)
-      (effects (font (size 1.27 1.27)) hide)
-    )
-    (property "LCSC Part #" "C25890" (at 133.35 124.46 0)
+    (property "Vendor PN" "C25744" (at 130.81 121.92 0)
+      (effects (font (size 1.27 1.27)) hide)
+    )
+    (property "LCSC Part #" "C25744" (at 133.35 124.46 0)
       (effects (font (size 1.27 1.27)) (justify left))
     )
@@
       (effects (font (size 1.27 1.27)) (justify left))
     )
-    (property "Value" "10uF/6,3V/0603" (at 130.81 32.385 0)
+    (property "Value" "10uF/10V/0603" (at 130.81 32.385 0)
       (effects (font (size 1.27 1.27)) (justify left))
     )
@@
       (effects (font (size 1.27 1.27)) hide)
     )
-    (property "Mfr PN" "CL10A106MQ8NNNC" (at 128.27 31.75 0)
+    (property "Mfr PN" "CL10A106KP8NNNC" (at 128.27 31.75 0)
       (effects (font (size 1.27 1.27)) hide)
     )
@@
       (effects (font (size 1.27 1.27)) hide)
     )
-    (property "LCSC Part #" "C1691" (at 130.81 37.465 0)
+    (property "LCSC Part #" "C19702" (at 130.81 37.465 0)
       (effects (font (size 1.27 1.27)) (justify left))
     )
@@
       (effects (font (size 1.27 1.27)) hide)
     )
-    (property "Vendor PN" "C1691" (at 128.27 31.75 0)
+    (property "Vendor PN" "C19702" (at 128.27 31.75 0)
       (effects (font (size 1.27 1.27)) hide)
     )
@@
       (effects (font (size 1.27 1.27)) (justify left))
     )
-    (property "Value" "0,1uF/16V/0402" (at 76.2 167.6462 0)
+    (property "Value" "0,1uF/50V/0402" (at 76.2 167.6462 0)
       (effects (font (size 1.27 1.27)) (justify left))
     )
@@
       (effects (font (size 1.27 1.27)) hide)
     )
-    (property "LCSC Part #" "C1525" (at 76.2 172.72 0)
+    (property "LCSC Part #" "C307331" (at 76.2 172.72 0)
       (effects (font (size 1.27 1.27)) (justify left))
     )
@@
       (effects (font (size 1.27 1.27)) hide)
     )
-    (property "Mfr PN" "CL05B104KO5NNNC" (at 73.66 166.37 0)
+    (property "Mfr PN" "CL05B104KB54PNC" (at 73.66 166.37 0)
       (effects (font (size 1.27 1.27)) hide)
     )
@@
       (effects (font (size 1.27 1.27)) hide)
     )
-    (property "Vendor PN" "C1525" (at 73.66 166.37 0)
+    (property "Vendor PN" "C307331" (at 73.66 166.37 0)
       (effects (font (size 1.27 1.27)) hide)
     )
@@
       (effects (font (size 1.27 1.27)) (justify left))
     )
-    (property "Value" "1uF/6,3V/0402" (at 231.14 43.1862 0)
+    (property "Value" "1uF/25V/0402" (at 231.14 43.1862 0)
       (effects (font (size 1.27 1.27)) (justify left))
     )
@@
       (effects (font (size 1.27 1.27)) hide)
     )
-    (property "LCSC Part #" "C107372" (at 231.14 48.26 0)
+    (property "LCSC Part #" "C52923" (at 231.14 48.26 0)
       (effects (font (size 1.27 1.27)) (justify left))
     )
@@
       (effects (font (size 1.27 1.27)) hide)
     )
-    (property "Mfr PN" "CL05A105KQ5NNNC" (at 228.6 43.18 0)
+    (property "Mfr PN" "CL05A105KA5NQNC" (at 228.6 43.18 0)
       (effects (font (size 1.27 1.27)) hide)
     )
@@
       (effects (font (size 1.27 1.27)) hide)
     )
-    (property "Vendor PN" "C107372" (at 228.6 43.18 0)
+    (property "Vendor PN" "C52923" (at 228.6 43.18 0)
       (effects (font (size 1.27 1.27)) hide)
     )
@@
       (effects (font (size 1.27 1.27)) (justify left))
     )
-    (property "Value" "0,1uF/16V/0402" (at 153.67 31.75 0)
+    (property "Value" "0,1uF/50V/0402" (at 153.67 31.75 0)
       (effects (font (size 1.27 1.27)) (justify left))
     )
@@
       (effects (font (size 1.27 1.27)) hide)
     )
-    (property "LCSC Part #" "C1525" (at 153.67 36.8238 0)
+    (property "LCSC Part #" "C307331" (at 153.67 36.8238 0)
       (effects (font (size 1.27 1.27)) (justify left))
     )
@@
       (effects (font (size 1.27 1.27)) hide)
     )
-    (property "Mfr PN" "CL05B104KO5NNNC" (at 151.13 31.75 0)
+    (property "Mfr PN" "CL05B104KB54PNC" (at 151.13 31.75 0)
       (effects (font (size 1.27 1.27)) hide)
     )
@@
       (effects (font (size 1.27 1.27)) hide)
     )
-    (property "Vendor PN" "C1525" (at 151.13 31.75 0)
+    (property "Vendor PN" "C307331" (at 151.13 31.75 0)
       (effects (font (size 1.27 1.27)) hide)
     )
@@
       (effects (font (size 1.27 1.27)) (justify left))
     )
-    (property "Value" "10uF/6,3V/0603" (at 133.35 131.445 0)
+    (property "Value" "10uF/10V/0603" (at 133.35 131.445 0)
       (effects (font (size 1.27 1.27)) (justify left))
     )
@@
       (effects (font (size 1.27 1.27)) hide)
     )
-    (property "Mfr PN" "CL10A106MQ8NNNC" (at 130.81 130.81 0)
+    (property "Mfr PN" "CL10A106KP8NNNC" (at 130.81 130.81 0)
       (effects (font (size 1.27 1.27)) hide)
     )
@@
       (effects (font (size 1.27 1.27)) hide)
     )
-    (property "LCSC Part #" "C1691" (at 133.35 136.525 0)
+    (property "LCSC Part #" "C19702" (at 133.35 136.525 0)
       (effects (font (size 1.27 1.27)) (justify left))
     )
@@
       (effects (font (size 1.27 1.27)) hide)
     )
-    (property "Vendor PN" "C1691" (at 130.81 130.81 0)
+    (property "Vendor PN" "C19702" (at 130.81 130.81 0)
       (effects (font (size 1.27 1.27)) hide)
     )
@@
       (effects (font (size 1.27 1.27)) (justify left))
     )
-    (property "Value" "470pF/16V/0402" (at 251.46 43.18 0)
+    (property "Value" "470pF/50V/0402" (at 251.46 43.18 0)
       (effects (font (size 1.27 1.27)) (justify left))
     )
@@
       (effects (font (size 1.27 1.27)) hide)
     )
-    (property "LCSC Part #" "C541379" (at 251.46 48.26 0)
-      (effects (font (size 1.27 1.27)) (justify left))
-    )
-    (property "Mfr" "Yageo" (at 248.92 43.18 0)
-      (effects (font (size 1.27 1.27)) hide)
-    )
-    (property "Mfr PN" "CC0402KRX7R7BB471" (at 248.92 43.18 0)
+    (property "LCSC Part #" "C1537" (at 251.46 48.26 0)
+      (effects (font (size 1.27 1.27)) (justify left))
+    )
+    (property "Mfr" "FH" (at 248.92 43.18 0)
+      (effects (font (size 1.27 1.27)) hide)
+    )
+    (property "Mfr PN" "0402B471K500NT" (at 248.92 43.18 0)
       (effects (font (size 1.27 1.27)) hide)
     )
@@
       (effects (font (size 1.27 1.27)) hide)
     )
-    (property "Vendor PN" "C541379" (at 248.92 43.18 0)
+    (property "Vendor PN" "C1537" (at 248.92 43.18 0)
       (effects (font (size 1.27 1.27)) hide)
     )
@@
       (effects (font (size 1.27 1.27)) (justify left) hide)
     )
-    (property "Datasheet" "http://ww1.microchip.com/downloads/en/DeviceDoc/8710a.pdf" (at 173.99 113.03 0)
+    (property "Datasheet" "~" (at 173.99 113.03 0)
       (effects (font (size 1.27 1.27)) hide)
     )
@@
       (effects (font (size 1.27 1.27)) (justify left))
     )
-    (property "Value" "0,1uF/16V/0402" (at 186.69 43.18 0)
+    (property "Value" "0,1uF/50V/0402" (at 186.69 43.18 0)
       (effects (font (size 1.27 1.27)) (justify left))
     )
@@
       (effects (font (size 1.27 1.27)) hide)
     )
-    (property "LCSC Part #" "C1525" (at 186.69 48.2538 0)
+    (property "LCSC Part #" "C307331" (at 186.69 48.2538 0)
       (effects (font (size 1.27 1.27)) (justify left))
     )
@@
       (effects (font (size 1.27 1.27)) hide)
     )
-    (property "Mfr PN" "CL05B104KO5NNNC" (at 184.15 43.18 0)
+    (property "Mfr PN" "CL05B104KB54PNC" (at 184.15 43.18 0)
       (effects (font (size 1.27 1.27)) hide)
     )
@@
       (effects (font (size 1.27 1.27)) hide)
     )
-    (property "Vendor PN" "C1525" (at 184.15 43.18 0)
-      (effects (font (size 1.27 1.27)) hide)
-    )
+    (property "Vendor PN" "C307331" (at 184.15 43.18 0)
+      (effects (font (size 1.27 1.27)) hide)
+    )

Commit message: Connectors rotated 180deg
Parts:
- D6: footprint Package_TO_SOT_SMD:SOT-23-5 -> Tales:SOT-23-5
Changed lines of the file:
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@@
       (effects (font (size 1.27 1.27)))
     )
-    (property "Footprint" "Package_TO_SOT_SMD:SOT-23-5" (at 254 91.44 0)
+    (property "Footprint" "Tales:SOT-23-5" (at 254 91.44 0)
       (effects (font (size 1.27 1.27)) hide)
     )
