File: V1/ESP-24v-32ch-V1-mcu.kicad_sch (KiCad schematic)
At the start: 12 parts, among them Q3 UMH3N, SW1 RESET, U3 CH340C, U4 ESP32-WROOM-32UE-N16

Commit message: Project rename
Other:
- title: ESP 16x 24VDC Input 16x External Relay Output Module -> ESP 32x 24VDC Input 32x 24VDC Output Module
Changed lines of the file:
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@@
   (paper "A4")
   (title_block
-    (title "ESP 16x 24VDC Input 16x External Relay Output Module")
-    (date "2022-10-20")
+    (title "ESP 32x 24VDC Input 32x 24VDC Output Module")
+    (date "2023-05-04")
     (rev "V1")
   )
@@
     (pin "1")
     (instances
-      (project "ESP-relay-32ch-V1"
+      (project "ESP-24v-32ch-V1"
         (path "/2bc5a21a-1d79-419d-a592-6852cc07b00a/f2a42251-1da5-495a-abaf-29698c5bb0fe"
           (reference "#PWR035") (unit 1)
@@
     (pin "2")
     (instances
-      (project "ESP-relay-32ch-V1"
+      (project "ESP-24v-32ch-V1"
         (path "/2bc5a21a-1d79-419d-a592-6852cc07b00a/f2a42251-1da5-495a-abaf-29698c5bb0fe"
           (reference "C13") (unit 1)
@@
     (pin "2")
     (instances
-      (project "ESP-relay-32ch-V1"
+      (project "ESP-24v-32ch-V1"
         (path "/2bc5a21a-1d79-419d-a592-6852cc07b00a/f2a42251-1da5-495a-abaf-29698c5bb0fe"
           (reference "R11") (unit 1)
@@
     (pin "1")
     (instances
-      (project "ESP-relay-32ch-V1"
+      (project "ESP-24v-32ch-V1"
         (path "/2bc5a21a-1d79-419d-a592-6852cc07b00a/f2a42251-1da5-495a-abaf-29698c5bb0fe"
           (reference "#PWR024") (unit 1)
@@
     (pin "5")
     (instances
-      (project "ESP-relay-32ch-V1"
+      (project "ESP-24v-32ch-V1"
         (path "/2bc5a21a-1d79-419d-a592-6852cc07b00a/f2a42251-1da5-495a-abaf-29698c5bb0fe"
           (reference "Q3") (unit 2)
@@
     (pin "2")
     (instances
-      (project "ESP-relay-32ch-V1"
+      (project "ESP-24v-32ch-V1"
         (path "/2bc5a21a-1d79-419d-a592-6852cc07b00a/f2a42251-1da5-495a-abaf-29698c5bb0fe"
           (reference "R12") (unit 1)
@@
     (pin "2")
     (instances
-      (project "ESP-relay-32ch-V1"
+      (project "ESP-24v-32ch-V1"
         (path "/2bc5a21a-1d79-419d-a592-6852cc07b00a/f2a42251-1da5-495a-abaf-29698c5bb0fe"
           (reference "C11") (unit 1)
@@
     (pin "5")
     (instances
-      (project "ESP-relay-32ch-V1"
+      (project "ESP-24v-32ch-V1"
         (path "/2bc5a21a-1d79-419d-a592-6852cc07b00a/f2a42251-1da5-495a-abaf-29698c5bb0fe"
           (reference "Q3") (unit 1)
@@
     (pin "1")
     (instances
-      (project "ESP-relay-32ch-V1"
+      (project "ESP-24v-32ch-V1"
         (path "/2bc5a21a-1d79-419d-a592-6852cc07b00a/f2a42251-1da5-495a-abaf-29698c5bb0fe"
           (reference "#PWR033") (unit 1)
@@
     (pin "2")
     (instances
-      (project "ESP-relay-32ch-V1"
+      (project "ESP-24v-32ch-V1"
         (path "/2bc5a21a-1d79-419d-a592-6852cc07b00a/f2a42251-1da5-495a-abaf-29698c5bb0fe"
           (reference "R14") (unit 1)
@@
     (pin "2")
     (instances
-      (project "ESP-relay-32ch-V1"
+      (project "ESP-24v-32ch-V1"
         (path "/2bc5a21a-1d79-419d-a592-6852cc07b00a/f2a42251-1da5-495a-abaf-29698c5bb0fe"
           (reference "SW1") (unit 1)
@@
     (pin "2")
     (instances
-      (project "ESP-relay-32ch-V1"
+      (project "ESP-24v-32ch-V1"
         (path "/2bc5a21a-1d79-419d-a592-6852cc07b00a/f2a42251-1da5-495a-abaf-29698c5bb0fe"
           (reference "R10") (unit 1)
@@
     (pin "1")
     (instances
-      (project "ESP-relay-32ch-V1"
+      (project "ESP-24v-32ch-V1"
         (path "/2bc5a21a-1d79-419d-a592-6852cc07b00a/f2a42251-1da5-495a-abaf-29698c5bb0fe"
           (reference "#PWR023") (unit 1)
@@
     (pin "1")
     (instances
-      (project "ESP-relay-32ch-V1"
+      (project "ESP-24v-32ch-V1"
         (path "/2bc5a21a-1d79-419d-a592-6852cc07b00a/f2a42251-1da5-495a-abaf-29698c5bb0fe"
           (reference "#PWR025") (unit 1)
@@
     (pin "1")
     (instances
-      (project "ESP-relay-32ch-V1"
+      (project "ESP-24v-32ch-V1"
         (path "/2bc5a21a-1d79-419d-a592-6852cc07b00a/f2a42251-1da5-495a-abaf-29698c5bb0fe"
           (reference "#PWR028") (unit 1)
@@
     (pin "9")
     (instances
-      (project "ESP-relay-32ch-V1"
+      (project "ESP-24v-32ch-V1"
         (path "/2bc5a21a-1d79-419d-a592-6852cc07b00a/f2a42251-1da5-495a-abaf-29698c5bb0fe"
           (reference "U3") (unit 1)
@@
     (pin "1")
     (instances
-      (project "ESP-relay-32ch-V1"
+      (project "ESP-24v-32ch-V1"
         (path "/2bc5a21a-1d79-419d-a592-6852cc07b00a/f2a42251-1da5-495a-abaf-29698c5bb0fe"
           (reference "#PWR026") (unit 1)
@@
     (pin "2")
     (instances
-      (project "ESP-relay-32ch-V1"
+      (project "ESP-24v-32ch-V1"
         (path "/2bc5a21a-1d79-419d-a592-6852cc07b00a/f2a42251-1da5-495a-abaf-29698c5bb0fe"
           (reference "R13") (unit 1)
@@
     (pin "9")
     (instances
-      (project "ESP-relay-32ch-V1"
+      (project "ESP-24v-32ch-V1"
         (path "/2bc5a21a-1d79-419d-a592-6852cc07b00a/f2a42251-1da5-495a-abaf-29698c5bb0fe"
           (reference "U4") (unit 1)
@@
     (pin "2")
     (instances
-      (project "ESP-relay-32ch-V1"
+      (project "ESP-24v-32ch-V1"
         (path "/2bc5a21a-1d79-419d-a592-6852cc07b00a/f2a42251-1da5-495a-abaf-29698c5bb0fe"
           (reference "C12") (unit 1)
@@
     (pin "1")
     (instances
-      (project "ESP-relay-32ch-V1"
+      (project "ESP-24v-32ch-V1"
         (path "/2bc5a21a-1d79-419d-a592-6852cc07b00a/f2a42251-1da5-495a-abaf-29698c5bb0fe"
           (reference "#PWR030") (unit 1)
@@
     (pin "1")
     (instances
-      (project "ESP-relay-32ch-V1"
+      (project "ESP-24v-32ch-V1"
         (path "/2bc5a21a-1d79-419d-a592-6852cc07b00a/f2a42251-1da5-495a-abaf-29698c5bb0fe"
           (reference "#PWR027") (unit 1)
@@
     (pin "1")
     (instances
-      (project "ESP-relay-32ch-V1"
+      (project "ESP-24v-32ch-V1"
         (path "/2bc5a21a-1d79-419d-a592-6852cc07b00a/f2a42251-1da5-495a-abaf-29698c5bb0fe"
           (reference "#PWR029") (unit 1)
@@
     (pin "1")
     (instances
-      (project "ESP-relay-32ch-V1"
+      (project "ESP-24v-32ch-V1"
         (path "/2bc5a21a-1d79-419d-a592-6852cc07b00a/f2a42251-1da5-495a-abaf-29698c5bb0fe"
           (reference "#PWR031") (unit 1)
@@
     (pin "1")
     (instances
-      (project "ESP-relay-32ch-V1"
+      (project "ESP-24v-32ch-V1"
         (path "/2bc5a21a-1d79-419d-a592-6852cc07b00a/f2a42251-1da5-495a-abaf-29698c5bb0fe"
           (reference "#PWR032") (unit 1)
@@
     (pin "1")
     (instances
-      (project "ESP-relay-32ch-V1"
+      (project "ESP-24v-32ch-V1"
         (path "/2bc5a21a-1d79-419d-a592-6852cc07b00a/f2a42251-1da5-495a-abaf-29698c5bb0fe"
           (reference "#PWR034") (unit 1)

Commit message: Dev
Parts:
- C11: value 10uF/6,3V/0603 -> 10uF/10V/0603; LCSC Part # C1691 -> C19702; Mfr PN CL10A106MQ8NNNC -> CL10A106KP8NNNC; Vendor PN C1691 -> C19702
- C13: value 1uF/10V/0603 -> 1uF/50V/0603; LCSC Part # C26413 -> C15849; Mfr PN CL10A105KP8NNNC -> CL10A105KB8NNNC; Vendor PN C26413 -> C15849
- R10, R11, R12: LCSC Part # C25890 -> C25744; Vendor PN C25890 -> C25744
Changed lines of the file:
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@@
       (effects (font (size 1.27 1.27)) (justify left))
     )
-    (property "Value" "1uF/10V/0603" (at 135.89 86.3662 0)
+    (property "Value" "1uF/50V/0603" (at 135.89 86.3662 0)
       (effects (font (size 1.27 1.27)) (justify left))
     )
@@
       (effects (font (size 1.27 1.27)) hide)
     )
-    (property "LCSC Part #" "C26413" (at 135.89 91.44 0)
+    (property "LCSC Part #" "C15849" (at 135.89 91.44 0)
       (effects (font (size 1.27 1.27)) (justify left))
     )
@@
       (effects (font (size 1.27 1.27)) hide)
     )
-    (property "Mfr PN" "CL10A105KP8NNNC" (at 133.35 86.36 0)
+    (property "Mfr PN" "CL10A105KB8NNNC" (at 133.35 86.36 0)
       (effects (font (size 1.27 1.27)) hide)
     )
@@
       (effects (font (size 1.27 1.27)) hide)
     )
-    (property "Vendor PN" "C26413" (at 133.35 86.36 0)
+    (property "Vendor PN" "C15849" (at 133.35 86.36 0)
       (effects (font (size 1.27 1.27)) hide)
     )
@@
       (effects (font (size 1.27 1.27)) hide)
     )
-    (property "Vendor PN" "C25890" (at 209.55 72.39 0)
-      (effects (font (size 1.27 1.27)) hide)
-    )
-    (property "LCSC Part #" "C25890" (at 207.01 72.39 0)
+    (property "Vendor PN" "C25744" (at 209.55 72.39 0)
+      (effects (font (size 1.27 1.27)) hide)
+    )
+    (property "LCSC Part #" "C25744" (at 207.01 72.39 0)
       (effects (font (size 1.27 1.27)) (justify right))
     )
@@
       (effects (font (size 1.27 1.27)) hide)
     )
-    (property "Datasheet" "http://rohmfs.rohm.com/en/products/databook/datasheet/discrete/transistor/digital/emh3t2r-e.pdf" (at 106.68 73.66 0)
+    (property "Datasheet" "~" (at 106.68 73.66 0)
       (effects (font (size 1.27 1.27)) hide)
     )
@@
       (effects (font (size 1.27 1.27)) hide)
     )
-    (property "Vendor PN" "C25890" (at 224.79 101.6 0)
-      (effects (font (size 1.27 1.27)) hide)
-    )
-    (property "LCSC Part #" "C25890" (at 227.33 106.68 0)
+    (property "Vendor PN" "C25744" (at 224.79 101.6 0)
+      (effects (font (size 1.27 1.27)) hide)
+    )
+    (property "LCSC Part #" "C25744" (at 227.33 106.68 0)
       (effects (font (size 1.27 1.27)) (justify left))
     )
@@
       (effects (font (size 1.27 1.27)) (justify left))
     )
-    (property "Value" "10uF/6,3V/0603" (at 24.13 60.96 0)
+    (property "Value" "10uF/10V/0603" (at 24.13 60.96 0)
       (effects (font (size 1.27 1.27)) (justify left))
     )
@@
       (effects (font (size 1.27 1.27)) hide)
     )
-    (property "Mfr PN" "CL10A106MQ8NNNC" (at 21.59 62.23 0)
+    (property "Mfr PN" "CL10A106KP8NNNC" (at 21.59 62.23 0)
       (effects (font (size 1.27 1.27)) hide)
     )
@@
       (effects (font (size 1.27 1.27)) hide)
     )
-    (property "Vendor PN" "C1691" (at 21.59 62.23 0)
-      (effects (font (size 1.27 1.27)) hide)
-    )
-    (property "LCSC Part #" "C1691" (at 24.13 66.04 0)
+    (property "Vendor PN" "C19702" (at 21.59 62.23 0)
+      (effects (font (size 1.27 1.27)) hide)
+    )
+    (property "LCSC Part #" "C19702" (at 24.13 66.04 0)
       (effects (font (size 1.27 1.27)) (justify left))
     )
@@
       (effects (font (size 1.27 1.27)) hide)
     )
-    (property "Datasheet" "http://rohmfs.rohm.com/en/products/databook/datasheet/discrete/transistor/digital/emh3t2r-e.pdf" (at 106.68 93.98 0)
+    (property "Datasheet" "~" (at 106.68 93.98 0)
       (effects (font (size 1.27 1.27)) hide)
     )
@@
       (effects (font (size 1.27 1.27)) hide)
     )
-    (property "Vendor PN" "C25890" (at 133.35 72.39 0)
-      (effects (font (size 1.27 1.27)) hide)
-    )
-    (property "LCSC Part #" "C25890" (at 135.89 72.39 0)
+    (property "Vendor PN" "C25744" (at 133.35 72.39 0)
+      (effects (font (size 1.27 1.27)) hide)
+    )
+    (property "LCSC Part #" "C25744" (at 135.89 72.39 0)
       (effects (font (size 1.27 1.27)) (justify left))
     )
@@
       (effects (font (size 1.27 1.27)) (justify left) hide)
     )
-    (property "Datasheet" "https://datasheet.lcsc.com/szlcsc/Jiangsu-Qin-Heng-CH340C_C84681.pdf" (at 54.61 66.04 0)
+    (property "Datasheet" "~" (at 54.61 66.04 0)
       (effects (font (size 1.27 1.27)) hide)
     )
@@
       (effects (font (size 1.27 1.27)) hide)
     )
-    (property "Datasheet" "https://www.espressif.com/sites/default/files/documentation/esp32-wroom-32d_esp32-wroom-32u_datasheet_en.pdf" (at 171.45 109.22 0)
-      (effects (font (size 1.27 1.27)) hide)
-    )
+    (property "Datasheet" "~" (at 171.45 109.22 0)
+      (effects (font (size 1.27 1.27)) hide)
+    )

Commit message: Connectors rotated 180deg
Parts:
- U3: footprint Package_SO:SOIC-16_3.9x9.9mm_P1.27mm -> Tales:SOIC-16_3.9x9.9mm_P1.27mm
Changed lines of the file:
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@@
       (effects (font (size 1.27 1.27)) (justify right))
     )
-    (property "Footprint" "Package_SO:SOIC-16_3.9x9.9mm_P1.27mm" (at 64.77 100.33 0)
+    (property "Footprint" "Tales:SOIC-16_3.9x9.9mm_P1.27mm" (at 64.77 100.33 0)
       (effects (font (size 1.27 1.27)) (justify left) hide)
     )

Commit message: Design optimization
Parts:
- SW1: footprint Button_Switch_SMD:SW_SPST_TL3342 -> Tales:SW_SPST_TL3342
Changed lines of the file:
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@@
       (effects (font (size 1.27 1.27)) (justify right))
     )
-    (property "Footprint" "Button_Switch_SMD:SW_SPST_TL3342" (at 120.65 111.76 0)
+    (property "Footprint" "Tales:SW_SPST_TL3342" (at 120.65 111.76 0)
       (effects (font (size 1.27 1.27)) hide)
     )
