File: V1/ESP-24v-32ch-V1-outputs-1.kicad_sch (KiCad schematic)
At the start: 80 parts, among them Q10 MMBT2222A/SOT-23-3, Q11 MMBT2222A/SOT-23-3, Q12 MMBT2222A/SOT-23-3, Q13 MMBT2222A/SOT-23-3, Q14 MMBT2222A/SOT-23-3, Q15 MMBT2222A/SOT-23-3, Q16 MMBT2222A/SOT-23-3, Q17 MMBT2222A/SOT-23-3, Q18 MMBT2222A/SOT-23-3, Q19 MMBT2222A/SOT-23-3, Q4 MMBT2222A/SOT-23-3, Q5 MMBT2222A/SOT-23-3, Q6 MMBT2222A/SOT-23-3, Q7 MMBT2222A/SOT-23-3, Q8 MMBT2222A/SOT-23-3, Q9 MMBT2222A/SOT-23-3

Commit message: Project rename
Parts:
- removed D39, D40, D41, D42, D43, D44, D45, D46, D47, D48, D49, D50, D51, D52, D53, D54: GREEN/0603, Tales:LED_0603_1608Metric, symbol Device:LED_Small
- removed R100, R103, R106, R109, R112, R115, R118, R121, R124, R79, R82, R85, R88, R91, R94, R97: 10k/62,5mW/0402, Tales:R_0402_1005Metric, symbol Device:R_US
- removed R101, R104, R107, R110, R113, R116, R119, R122, R125, R80, R83, R86, R89, R92, R95, R98: 1k/62,5mW/0402, Tales:R_0402_1005Metric, symbol Device:R_US
- removed R102, R105, R108, R111, R114, R117, R120, R123, R126, R81, R84, R87, R90, R93, R96, R99: 5,6k/0,1W/0603, Tales:R_0603_1608Metric, symbol Device:R_US
- added D71, D72, D73, D74, D75, D76, D77, D78, D79, D80, D81, D82, D83, D84, D85, D86: GREEN/0603, Tales:LED_0603_1608Metric, symbol Device:LED_Small
- added R131, R132, R133, R134, R143, R144, R145, R146, R155, R156, R157, R158, R167, R168, R169, R170: 10k/62,5mW/0402, Tales:R_0402_1005Metric, symbol Device:R_US
- added R135, R136, R137, R138, R147, R148, R149, R150, R159, R160, R161, R162, R171, R172, R173, R174: 1k/62,5mW/0402, Tales:R_0402_1005Metric, symbol Device:R_US
- added R139, R140, R141, R142, R151, R152, R153, R154, R163, R164, R165, R166, R175, R176, R177, R178: 5,6k/0,1W/0603, Tales:R_0603_1608Metric, symbol Device:R_US
Connections:
- net +24V: now also R139.1, R140.1, R141.1, R142.1, R151.1, R152.1, R153.1, R154.1, R163.1, R164.1, R165.1, R166.1, R175.1, R176.1, R177.1, R178.1
- net GND: now also R131.2, R132.2, R133.2, R134.2, R143.2, R144.2, R145.2, R146.2, R155.2, R156.2, R157.2, R158.2, R167.2, R168.2, R169.2, R170.2
- net at Q15.1 (B): now also R162.1
- net at Q4.1 (B): now also R135.1
- net at Q19.1 (B): now also R174.1
- net at Q9.1 (B): now also R148.1
- net at Q10.1 (B): now also R149.1
- net at Q18.1 (B): now also R173.1
- net at Q5.1 (B): now also R136.1
- net at Q7.1 (B): now also R138.1
- net at Q6.1 (B): now also R137.1
- net at Q16.1 (B): now also R171.1
- net at Q13.1 (B): now also R160.1
- net at Q11.1 (B): now also R150.1
- net at Q14.1 (B): now also R161.1
- net at Q8.1 (B): now also R147.1
- net at Q12.1 (B): now also R159.1
- net at Q17.1 (B): now also R172.1
- net J10-OUT17 renamed J8-OUT1
- net J8-OUT1: now also D71.1 (K)
- net J10-OUT18 renamed J8-OUT2
- net J8-OUT2: now also D72.1 (K)
- net J10-OUT19 renamed J8-OUT3
- net J8-OUT3: now also D73.1 (K)
- net J10-OUT20 renamed J8-OUT4
- net J8-OUT4: now also D74.1 (K)
- net J10-OUT21 renamed J8-OUT5
- net J8-OUT5: now also D75.1 (K)
- net J10-OUT22 renamed J8-OUT6
- net J8-OUT6: now also D76.1 (K)
- net J10-OUT23 renamed J8-OUT7
- net J8-OUT7: now also D77.1 (K)
- net J10-OUT24 renamed J8-OUT8
- net J8-OUT8: now also D78.1 (K)
- net J11-OUT25 renamed J9-OUT9
- net J9-OUT9: now also D79.1 (K)
- net J11-OUT26 renamed J9-OUT10
- net J9-OUT10: now also D80.1 (K)
- net J11-OUT27 renamed J9-OUT11
- net J9-OUT11: now also D81.1 (K)
- net J11-OUT28 renamed J9-OUT12
- net J9-OUT12: now also D82.1 (K)
- net J11-OUT29 renamed J9-OUT13
- net J9-OUT13: now also D83.1 (K)
- net J11-OUT30 renamed J9-OUT14
- net J9-OUT14: now also D84.1 (K)
- net J11-OUT31 renamed J9-OUT15
- net J9-OUT15: now also D85.1 (K)
- net J11-OUT32 renamed J9-OUT16
- net J9-OUT16: now also D86.1 (K)
- new net: D84.2 (A), R176.2
- new net: D73.2 (A), R141.2
- new net: D83.2 (A), R175.2
- new net: D86.2 (A), R178.2
- new net: D71.2 (A), R139.2
- new net: D76.2 (A), R152.2
- new net: D82.2 (A), R166.2
- new net: D80.2 (A), R164.2
- new net: D77.2 (A), R153.2
- new net: D79.2 (A), R163.2
- new net: D75.2 (A), R151.2
- new net: D78.2 (A), R154.2
- new net: D74.2 (A), R142.2
- new net: D85.2 (A), R177.2
- new net: D72.2 (A), R140.2
- new net: D81.2 (A), R165.2
- new net OUT1: R131.1, R135.2
- new net OUT10: R156.1, R160.2
- new net OUT11: R157.1, R161.2
- new net OUT12: R158.1, R162.2
- new net OUT13: R167.1, R171.2
- new net OUT14: R168.1, R172.2
- new net OUT15: R169.1, R173.2
- new net OUT16: R170.1, R174.2
- new net OUT2: R132.1, R136.2
- new net OUT3: R133.1, R137.2
- new net OUT4: R134.1, R138.2
- new net OUT5: R143.1, R147.2
- new net OUT6: R144.1, R148.2
- new net OUT7: R145.1, R149.2
- new net OUT8: R146.1, R150.2
- new net OUT9: R155.1, R159.2
Other:
- title: ESP 16x 24VDC Input 16x External Relay Output Module -> ESP 32x 24VDC Input 32x 24VDC Output Module

Commit message: Dev
Parts:
- R131, R132, R133, R134, R143, R144, R145, R146, R155, R156, R157, R158, R167, R168, R169, R170: LCSC Part # C25890 -> C25744; Vendor PN C25890 -> C25744
Changed lines of the file:
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@@
       (effects (font (size 1.27 1.27)) hide)
     )
-    (property "Vendor PN" "C25890" (at 93.98 157.48 0)
+    (property "Vendor PN" "C25744" (at 93.98 157.48 0)
       (effects (font (size 1.27 1.27)) hide)
     )
-    (property "LCSC Part #" "C25890" (at 96.52 162.56 0)
+    (property "LCSC Part #" "C25744" (at 96.52 162.56 0)
       (effects (font (size 1.27 1.27)) (justify left))
     )
@@
       (effects (font (size 1.27 1.27)) hide)
     )
-    (property "Vendor PN" "C25890" (at 158.75 45.72 0)
+    (property "Vendor PN" "C25744" (at 158.75 45.72 0)
       (effects (font (size 1.27 1.27)) hide)
     )
-    (property "LCSC Part #" "C25890" (at 161.29 52.07 0)
+    (property "LCSC Part #" "C25744" (at 161.29 52.07 0)
       (effects (font (size 1.27 1.27)) (justify left))
     )
@@
       (effects (font (size 1.27 1.27)) hide)
     )
-    (property "Vendor PN" "C25890" (at 93.98 83.82 0)
+    (property "Vendor PN" "C25744" (at 93.98 83.82 0)
       (effects (font (size 1.27 1.27)) hide)
     )
-    (property "LCSC Part #" "C25890" (at 96.52 88.9 0)
+    (property "LCSC Part #" "C25744" (at 96.52 88.9 0)
       (effects (font (size 1.27 1.27)) (justify left))
     )
@@
       (effects (font (size 1.27 1.27)) hide)
     )
-    (property "Vendor PN" "C25890" (at 222.25 120.65 0)
+    (property "Vendor PN" "C25744" (at 222.25 120.65 0)
       (effects (font (size 1.27 1.27)) hide)
     )
-    (property "LCSC Part #" "C25890" (at 224.79 125.73 0)
+    (property "LCSC Part #" "C25744" (at 224.79 125.73 0)
       (effects (font (size 1.27 1.27)) (justify left))
     )
@@
       (effects (font (size 1.27 1.27)) hide)
     )
-    (property "Vendor PN" "C25890" (at 158.75 156.21 0)
+    (property "Vendor PN" "C25744" (at 158.75 156.21 0)
       (effects (font (size 1.27 1.27)) hide)
     )
-    (property "LCSC Part #" "C25890" (at 161.29 162.56 0)
+    (property "LCSC Part #" "C25744" (at 161.29 162.56 0)
       (effects (font (size 1.27 1.27)) (justify left))
     )
@@
       (effects (font (size 1.27 1.27)) hide)
     )
-    (property "Vendor PN" "C25890" (at 93.98 120.65 0)
+    (property "Vendor PN" "C25744" (at 93.98 120.65 0)
       (effects (font (size 1.27 1.27)) hide)
     )
-    (property "LCSC Part #" "C25890" (at 96.52 125.73 0)
+    (property "LCSC Part #" "C25744" (at 96.52 125.73 0)
       (effects (font (size 1.27 1.27)) (justify left))
     )
@@
       (effects (font (size 1.27 1.27)) hide)
     )
-    (property "Vendor PN" "C25890" (at 222.25 46.99 0)
+    (property "Vendor PN" "C25744" (at 222.25 46.99 0)
       (effects (font (size 1.27 1.27)) hide)
     )
-    (property "LCSC Part #" "C25890" (at 224.79 52.07 0)
+    (property "LCSC Part #" "C25744" (at 224.79 52.07 0)
       (effects (font (size 1.27 1.27)) (justify left))
     )
@@
       (effects (font (size 1.27 1.27)) hide)
     )
-    (property "Vendor PN" "C25890" (at 29.21 82.55 0)
+    (property "Vendor PN" "C25744" (at 29.21 82.55 0)
       (effects (font (size 1.27 1.27)) hide)
     )
-    (property "LCSC Part #" "C25890" (at 31.75 88.9 0)
+    (property "LCSC Part #" "C25744" (at 31.75 88.9 0)
       (effects (font (size 1.27 1.27)) (justify left))
     )
@@
       (effects (font (size 1.27 1.27)) hide)
     )
-    (property "Vendor PN" "C25890" (at 29.21 156.21 0)
+    (property "Vendor PN" "C25744" (at 29.21 156.21 0)
       (effects (font (size 1.27 1.27)) hide)
     )
-    (property "LCSC Part #" "C25890" (at 31.75 162.56 0)
+    (property "LCSC Part #" "C25744" (at 31.75 162.56 0)
       (effects (font (size 1.27 1.27)) (justify left))
     )
@@
       (effects (font (size 1.27 1.27)) hide)
     )
-    (property "Vendor PN" "C25890" (at 93.98 46.99 0)
+    (property "Vendor PN" "C25744" (at 93.98 46.99 0)
       (effects (font (size 1.27 1.27)) hide)
     )
-    (property "LCSC Part #" "C25890" (at 96.52 52.07 0)
+    (property "LCSC Part #" "C25744" (at 96.52 52.07 0)
       (effects (font (size 1.27 1.27)) (justify left))
     )
@@
       (effects (font (size 1.27 1.27)) hide)
     )
-    (property "Vendor PN" "C25890" (at 158.75 119.38 0)
+    (property "Vendor PN" "C25744" (at 158.75 119.38 0)
       (effects (font (size 1.27 1.27)) hide)
     )
-    (property "LCSC Part #" "C25890" (at 161.29 123.19 0)
+    (property "LCSC Part #" "C25744" (at 161.29 123.19 0)
       (effects (font (size 1.27 1.27)) (justify left))
     )
@@
       (effects (font (size 1.27 1.27)) hide)
     )
-    (property "Vendor PN" "C25890" (at 222.25 157.48 0)
+    (property "Vendor PN" "C25744" (at 222.25 157.48 0)
       (effects (font (size 1.27 1.27)) hide)
     )
-    (property "LCSC Part #" "C25890" (at 224.79 162.56 0)
+    (property "LCSC Part #" "C25744" (at 224.79 162.56 0)
       (effects (font (size 1.27 1.27)) (justify left))
     )
@@
       (effects (font (size 1.27 1.27)) hide)
     )
-    (property "Vendor PN" "C25890" (at 158.75 82.55 0)
+    (property "Vendor PN" "C25744" (at 158.75 82.55 0)
       (effects (font (size 1.27 1.27)) hide)
     )
-    (property "LCSC Part #" "C25890" (at 161.29 88.9 0)
+    (property "LCSC Part #" "C25744" (at 161.29 88.9 0)
       (effects (font (size 1.27 1.27)) (justify left))
     )
@@
       (effects (font (size 1.27 1.27)) hide)
     )
-    (property "Vendor PN" "C25890" (at 222.25 83.82 0)
+    (property "Vendor PN" "C25744" (at 222.25 83.82 0)
       (effects (font (size 1.27 1.27)) hide)
     )
-    (property "LCSC Part #" "C25890" (at 224.79 88.9 0)
+    (property "LCSC Part #" "C25744" (at 224.79 88.9 0)
       (effects (font (size 1.27 1.27)) (justify left))
     )
@@
       (effects (font (size 1.27 1.27)) hide)
     )
-    (property "Vendor PN" "C25890" (at 29.21 45.72 0)
+    (property "Vendor PN" "C25744" (at 29.21 45.72 0)
       (effects (font (size 1.27 1.27)) hide)
     )
-    (property "LCSC Part #" "C25890" (at 31.75 52.07 0)
+    (property "LCSC Part #" "C25744" (at 31.75 52.07 0)
       (effects (font (size 1.27 1.27)) (justify left))
     )
@@
       (effects (font (size 1.27 1.27)) hide)
     )
-    (property "Vendor PN" "C25890" (at 29.21 119.38 0)
+    (property "Vendor PN" "C25744" (at 29.21 119.38 0)
       (effects (font (size 1.27 1.27)) hide)
     )
-    (property "LCSC Part #" "C25890" (at 31.75 123.19 0)
+    (property "LCSC Part #" "C25744" (at 31.75 123.19 0)
       (effects (font (size 1.27 1.27)) (justify left))
     )

Commit message: Renamed to lowercase
Parts:
- renumbered D84 to D100, D85 to D101, D86 to D102, D71 to D87, D72 to D88, D73 to D89, D74 to D90, D75 to D91, D76 to D92, D77 to D93, D78 to D94, D79 to D95, D80 to D96, D81 to D97, D82 to D98, D83 to D99, Q4 to Q20, Q5 to Q21, Q6 to Q22, Q7 to Q23, Q8 to Q24, Q9 to Q25, Q10 to Q26, Q11 to Q27, Q12 to Q28, Q13 to Q29, Q14 to Q30, Q15 to Q31, Q16 to Q32, Q17 to Q33, Q18 to Q34, Q19 to Q35, R131 to R179, R132 to R180, R133 to R181, R134 to R182, R135 to R183, R136 to R184, R137 to R185, R138 to R186, R139 to R187, R140 to R188, R141 to R189, R142 to R190, R143 to R191, R144 to R192, R145 to R193, R146 to R194, R147 to R195, R148 to R196, R149 to R197, R150 to R198, R151 to R199, R152 to R200, R153 to R201, R154 to R202, R155 to R203, R156 to R204, R157 to R205, R158 to R206, R159 to R207, R160 to R208, R161 to R209, R162 to R210, R163 to R211, R164 to R212, R165 to R213, R166 to R214, R167 to R215, R168 to R216, R169 to R217, R170 to R218, R171 to R219, R172 to R220, R173 to R221, R174 to R222, R175 to R223, R176 to R224, R177 to R225, R178 to R226
