File: V1/ESP-24v-32ch-V1-outputs-2.kicad_sch (KiCad schematic)
At the start: 80 parts, among them Q10 MMBT2222A/SOT-23-3, Q11 MMBT2222A/SOT-23-3, Q12 MMBT2222A/SOT-23-3, Q13 MMBT2222A/SOT-23-3, Q14 MMBT2222A/SOT-23-3, Q15 MMBT2222A/SOT-23-3, Q16 MMBT2222A/SOT-23-3, Q17 MMBT2222A/SOT-23-3, Q18 MMBT2222A/SOT-23-3, Q19 MMBT2222A/SOT-23-3, Q4 MMBT2222A/SOT-23-3, Q5 MMBT2222A/SOT-23-3, Q6 MMBT2222A/SOT-23-3, Q7 MMBT2222A/SOT-23-3, Q8 MMBT2222A/SOT-23-3, Q9 MMBT2222A/SOT-23-3

Commit message: Project rename
Parts:
- removed D71, D72, D73, D74, D75, D76, D77, D78, D79, D80, D81, D82, D83, D84, D85, D86: GREEN/0603, Tales:LED_0603_1608Metric, symbol Device:LED_Small
- removed R131, R132, R133, R134, R143, R144, R145, R146, R155, R156, R157, R158, R167, R168, R169, R170: 10k/62,5mW/0402, Tales:R_0402_1005Metric, symbol Device:R_US
- removed R135, R136, R137, R138, R147, R148, R149, R150, R159, R160, R161, R162, R171, R172, R173, R174: 1k/62,5mW/0402, Tales:R_0402_1005Metric, symbol Device:R_US
- removed R139, R140, R141, R142, R151, R152, R153, R154, R163, R164, R165, R166, R175, R176, R177, R178: 5,6k/0,1W/0603, Tales:R_0603_1608Metric, symbol Device:R_US
- added D39, D40, D41, D42, D43, D44, D45, D46, D47, D48, D49, D50, D51, D52, D53, D54: GREEN/0603, Tales:LED_0603_1608Metric, symbol Device:LED_Small
- added R100, R103, R106, R109, R112, R115, R118, R121, R124, R79, R82, R85, R88, R91, R94, R97: 10k/62,5mW/0402, Tales:R_0402_1005Metric, symbol Device:R_US
- added R101, R104, R107, R110, R113, R116, R119, R122, R125, R80, R83, R86, R89, R92, R95, R98: 1k/62,5mW/0402, Tales:R_0402_1005Metric, symbol Device:R_US
- added R102, R105, R108, R111, R114, R117, R120, R123, R126, R81, R84, R87, R90, R93, R96, R99: 5,6k/0,1W/0603, Tales:R_0603_1608Metric, symbol Device:R_US
Connections:
- net +24V: now also R102.1, R105.1, R108.1, R111.1, R114.1, R117.1, R120.1, R123.1, R126.1, R81.1, R84.1, R87.1, R90.1, R93.1, R96.1, R99.1
- net GND: now also R100.2, R103.2, R106.2, R109.2, R112.2, R115.2, R118.2, R121.2, R124.2, R79.2, R82.2, R85.2, R88.2, R91.2, R94.2, R97.2
- net at Q12.1 (B): now also R104.1
- net at Q19.1 (B): now also R125.1
- net at Q17.1 (B): now also R119.1
- net at Q8.1 (B): now also R92.1
- net at Q9.1 (B): now also R95.1
- net at Q5.1 (B): now also R83.1
- net at Q14.1 (B): now also R110.1
- net at Q16.1 (B): now also R116.1
- net at Q10.1 (B): now also R98.1
- net at Q13.1 (B): now also R107.1
- net at Q15.1 (B): now also R113.1
- net at Q7.1 (B): now also R89.1
- net at Q6.1 (B): now also R86.1
- net at Q4.1 (B): now also R80.1
- net at Q18.1 (B): now also R122.1
- net at Q11.1 (B): now also R101.1
- net J8-OUT1 renamed J10-OUT17
- net J10-OUT17: now also D39.1 (K)
- net J8-OUT2 renamed J10-OUT18
- net J10-OUT18: now also D40.1 (K)
- net J8-OUT3 renamed J10-OUT19
- net J10-OUT19: now also D41.1 (K)
- net J8-OUT4 renamed J10-OUT20
- net J10-OUT20: now also D42.1 (K)
- net J8-OUT5 renamed J10-OUT21
- net J10-OUT21: now also D43.1 (K)
- net J8-OUT6 renamed J10-OUT22
- net J10-OUT22: now also D44.1 (K)
- net J8-OUT7 renamed J10-OUT23
- net J10-OUT23: now also D45.1 (K)
- net J8-OUT8 renamed J10-OUT24
- net J10-OUT24: now also D46.1 (K)
- net J9-OUT10 renamed J11-OUT26
- net J11-OUT26: now also D48.1 (K)
- net J9-OUT11 renamed J11-OUT27
- net J11-OUT27: now also D49.1 (K)
- net J9-OUT12 renamed J11-OUT28
- net J11-OUT28: now also D50.1 (K)
- net J9-OUT13 renamed J11-OUT29
- net J11-OUT29: now also D51.1 (K)
- net J9-OUT14 renamed J11-OUT30
- net J11-OUT30: now also D52.1 (K)
- net J9-OUT15 renamed J11-OUT31
- net J11-OUT31: now also D53.1 (K)
- net J9-OUT16 renamed J11-OUT32
- net J11-OUT32: now also D54.1 (K)
- net J9-OUT9 renamed J11-OUT25
- net J11-OUT25: now also D47.1 (K)
- new net: D54.2 (A), R126.2
- new net: D43.2 (A), R93.2
- new net: D50.2 (A), R114.2
- new net: D46.2 (A), R102.2
- new net: D45.2 (A), R99.2
- new net: D49.2 (A), R111.2
- new net: D40.2 (A), R84.2
- new net: D53.2 (A), R123.2
- new net: D48.2 (A), R108.2
- new net: D44.2 (A), R96.2
- new net: D51.2 (A), R117.2
- new net: D42.2 (A), R90.2
- new net: D52.2 (A), R120.2
- new net: D39.2 (A), R81.2
- new net: D47.2 (A), R105.2
- new net: D41.2 (A), R87.2
- new net OUT17: R79.1, R80.2
- new net OUT18: R82.1, R83.2
- new net OUT19: R85.1, R86.2
- new net OUT20: R88.1, R89.2
- new net OUT21: R91.1, R92.2
- new net OUT22: R94.1, R95.2
- new net OUT23: R97.1, R98.2
- new net OUT24: R100.1, R101.2
- new net OUT25: R103.1, R104.2
- new net OUT26: R106.1, R107.2
- new net OUT27: R109.1, R110.2
- new net OUT28: R112.1, R113.2
- new net OUT29: R115.1, R116.2
- new net OUT30: R118.1, R119.2
- new net OUT31: R121.1, R122.2
- new net OUT32: R124.1, R125.2
Other:
- title: ESP 16x 24VDC Input 16x External Relay Output Module -> ESP 32x 24VDC Input 32x 24VDC Output Module

Commit message: Dev
Parts:
- R100, R103, R106, R109, R112, R115, R118, R121, R124, R79, R82, R85, R88, R91, R94, R97: LCSC Part # C25890 -> C25744; Vendor PN C25890 -> C25744
Changed lines of the file:
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@@
       (effects (font (size 1.27 1.27)) hide)
     )
-    (property "Vendor PN" "C25890" (at 158.75 119.38 0)
+    (property "Vendor PN" "C25744" (at 158.75 119.38 0)
       (effects (font (size 1.27 1.27)) hide)
     )
-    (property "LCSC Part #" "C25890" (at 161.29 123.19 0)
+    (property "LCSC Part #" "C25744" (at 161.29 123.19 0)
       (effects (font (size 1.27 1.27)) (justify left))
     )
@@
       (effects (font (size 1.27 1.27)) hide)
     )
-    (property "Vendor PN" "C25890" (at 222.25 157.48 0)
+    (property "Vendor PN" "C25744" (at 222.25 157.48 0)
       (effects (font (size 1.27 1.27)) hide)
     )
-    (property "LCSC Part #" "C25890" (at 224.79 162.56 0)
+    (property "LCSC Part #" "C25744" (at 224.79 162.56 0)
       (effects (font (size 1.27 1.27)) (justify left))
     )
@@
       (effects (font (size 1.27 1.27)) hide)
     )
-    (property "Vendor PN" "C25890" (at 29.21 119.38 0)
+    (property "Vendor PN" "C25744" (at 29.21 119.38 0)
       (effects (font (size 1.27 1.27)) hide)
     )
-    (property "LCSC Part #" "C25890" (at 31.75 123.19 0)
+    (property "LCSC Part #" "C25744" (at 31.75 123.19 0)
       (effects (font (size 1.27 1.27)) (justify left))
     )
@@
       (effects (font (size 1.27 1.27)) hide)
     )
-    (property "Vendor PN" "C25890" (at 29.21 45.72 0)
+    (property "Vendor PN" "C25744" (at 29.21 45.72 0)
       (effects (font (size 1.27 1.27)) hide)
     )
-    (property "LCSC Part #" "C25890" (at 31.75 52.07 0)
+    (property "LCSC Part #" "C25744" (at 31.75 52.07 0)
       (effects (font (size 1.27 1.27)) (justify left))
     )
@@
       (effects (font (size 1.27 1.27)) hide)
     )
-    (property "Vendor PN" "C25890" (at 222.25 83.82 0)
+    (property "Vendor PN" "C25744" (at 222.25 83.82 0)
       (effects (font (size 1.27 1.27)) hide)
     )
-    (property "LCSC Part #" "C25890" (at 224.79 88.9 0)
+    (property "LCSC Part #" "C25744" (at 224.79 88.9 0)
       (effects (font (size 1.27 1.27)) (justify left))
     )
@@
       (effects (font (size 1.27 1.27)) hide)
     )
-    (property "Vendor PN" "C25890" (at 29.21 82.55 0)
+    (property "Vendor PN" "C25744" (at 29.21 82.55 0)
       (effects (font (size 1.27 1.27)) hide)
     )
-    (property "LCSC Part #" "C25890" (at 31.75 88.9 0)
+    (property "LCSC Part #" "C25744" (at 31.75 88.9 0)
       (effects (font (size 1.27 1.27)) (justify left))
     )
@@
       (effects (font (size 1.27 1.27)) hide)
     )
-    (property "Vendor PN" "C25890" (at 29.21 156.21 0)
+    (property "Vendor PN" "C25744" (at 29.21 156.21 0)
       (effects (font (size 1.27 1.27)) hide)
     )
-    (property "LCSC Part #" "C25890" (at 31.75 162.56 0)
+    (property "LCSC Part #" "C25744" (at 31.75 162.56 0)
       (effects (font (size 1.27 1.27)) (justify left))
     )
@@
       (effects (font (size 1.27 1.27)) hide)
     )
-    (property "Vendor PN" "C25890" (at 158.75 45.72 0)
+    (property "Vendor PN" "C25744" (at 158.75 45.72 0)
       (effects (font (size 1.27 1.27)) hide)
     )
-    (property "LCSC Part #" "C25890" (at 161.29 52.07 0)
+    (property "LCSC Part #" "C25744" (at 161.29 52.07 0)
       (effects (font (size 1.27 1.27)) (justify left))
     )
@@
       (effects (font (size 1.27 1.27)) hide)
     )
-    (property "Vendor PN" "C25890" (at 93.98 157.48 0)
+    (property "Vendor PN" "C25744" (at 93.98 157.48 0)
       (effects (font (size 1.27 1.27)) hide)
     )
-    (property "LCSC Part #" "C25890" (at 96.52 162.56 0)
+    (property "LCSC Part #" "C25744" (at 96.52 162.56 0)
       (effects (font (size 1.27 1.27)) (justify left))
     )
@@
       (effects (font (size 1.27 1.27)) hide)
     )
-    (property "Vendor PN" "C25890" (at 158.75 82.55 0)
+    (property "Vendor PN" "C25744" (at 158.75 82.55 0)
       (effects (font (size 1.27 1.27)) hide)
     )
-    (property "LCSC Part #" "C25890" (at 161.29 88.9 0)
+    (property "LCSC Part #" "C25744" (at 161.29 88.9 0)
       (effects (font (size 1.27 1.27)) (justify left))
     )
@@
       (effects (font (size 1.27 1.27)) hide)
     )
-    (property "Vendor PN" "C25890" (at 158.75 156.21 0)
+    (property "Vendor PN" "C25744" (at 158.75 156.21 0)
       (effects (font (size 1.27 1.27)) hide)
     )
-    (property "LCSC Part #" "C25890" (at 161.29 162.56 0)
+    (property "LCSC Part #" "C25744" (at 161.29 162.56 0)
       (effects (font (size 1.27 1.27)) (justify left))
     )
@@
       (effects (font (size 1.27 1.27)) hide)
     )
-    (property "Vendor PN" "C25890" (at 222.25 120.65 0)
+    (property "Vendor PN" "C25744" (at 222.25 120.65 0)
       (effects (font (size 1.27 1.27)) hide)
     )
-    (property "LCSC Part #" "C25890" (at 224.79 125.73 0)
+    (property "LCSC Part #" "C25744" (at 224.79 125.73 0)
       (effects (font (size 1.27 1.27)) (justify left))
     )
@@
       (effects (font (size 1.27 1.27)) hide)
     )
-    (property "Vendor PN" "C25890" (at 93.98 120.65 0)
+    (property "Vendor PN" "C25744" (at 93.98 120.65 0)
       (effects (font (size 1.27 1.27)) hide)
     )
-    (property "LCSC Part #" "C25890" (at 96.52 125.73 0)
+    (property "LCSC Part #" "C25744" (at 96.52 125.73 0)
       (effects (font (size 1.27 1.27)) (justify left))
     )
@@
       (effects (font (size 1.27 1.27)) hide)
     )
-    (property "Vendor PN" "C25890" (at 93.98 46.99 0)
+    (property "Vendor PN" "C25744" (at 93.98 46.99 0)
       (effects (font (size 1.27 1.27)) hide)
     )
-    (property "LCSC Part #" "C25890" (at 96.52 52.07 0)
+    (property "LCSC Part #" "C25744" (at 96.52 52.07 0)
       (effects (font (size 1.27 1.27)) (justify left))
     )
@@
       (effects (font (size 1.27 1.27)) hide)
     )
-    (property "Vendor PN" "C25890" (at 93.98 83.82 0)
+    (property "Vendor PN" "C25744" (at 93.98 83.82 0)
       (effects (font (size 1.27 1.27)) hide)
     )
-    (property "LCSC Part #" "C25890" (at 96.52 88.9 0)
+    (property "LCSC Part #" "C25744" (at 96.52 88.9 0)
       (effects (font (size 1.27 1.27)) (justify left))
     )
@@
       (effects (font (size 1.27 1.27)) hide)
     )
-    (property "Vendor PN" "C25890" (at 222.25 46.99 0)
+    (property "Vendor PN" "C25744" (at 222.25 46.99 0)
       (effects (font (size 1.27 1.27)) hide)
     )
-    (property "LCSC Part #" "C25890" (at 224.79 52.07 0)
+    (property "LCSC Part #" "C25744" (at 224.79 52.07 0)
       (effects (font (size 1.27 1.27)) (justify left))
     )
