File: V1/ESP-24v-32ch-V1-power.kicad_sch (KiCad schematic)
At the start: 34 parts, among them J10 USB, J9 VIN, Q1 WPM2015-3/TR, Q2 LMUN2211LT1G, U1 SY8089A1AAC, U2 TX4138

Commit message: Project rename
Other:
- title: ESP 16x 24VDC Input 16x External Relay Output Module -> ESP 32x 24VDC Input 32x 24VDC Output Module

Commit message: Dev
Parts:
- C1, C5: value 10uF/16V/1206 -> 10uF/50V/1206; LCSC Part # C1849 -> C13585; Mfr PN CL31A106KOHNNNE -> CL31A106KBHNNNE; Vendor PN C1849 -> C13585
- C6, C9: value 10uF/6,3V/0603 -> 10uF/10V/0603; LCSC Part # C1691 -> C19702; Mfr PN CL10A106MQ8NNNC -> CL10A106KP8NNNC; Vendor PN C1691 -> C19702
- R6: LCSC Part # C25890 -> C25744; Vendor PN C25890 -> C25744
Other:
- note added: "R1"
- note added: "R2"
- note added: "RH"
- note added: "RL"
- note added: "R_{2} = R_{1}/(V_{OUT} / 0,805 - 1) V_{OUT} = (R_{1} / R_{2}) + 1) * 0,805 V_{OUT} = (300k / 52,3k + 1) * 0,805 V_{OUT} = 5,42V"
- note added: "R_{H} = (V_{OUT} - 0,6V) * R_{L} / 0,6V V_{OUT} = (0,6 * R_{H} / R_{L}) + 0,6 V_{OUT} = (0,6 * 100k/22,1k) +0,6 V_{OUT} = 3,31V"
- moved on the sheet: C8, R8, R9

Commit message: Connectors rotated 180deg
Parts:
- L3: footprint Inductor_SMD:L_0805_2012Metric -> Tales:L_0805_2012Metric
Changed lines of the file:
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@@
       (effects (font (size 1.27 1.27)))
     )
-    (property "Footprint" "Inductor_SMD:L_0805_2012Metric" (at 246.38 124.46 0)
+    (property "Footprint" "Tales:L_0805_2012Metric" (at 246.38 124.46 0)
       (effects (font (size 1.27 1.27)) hide)
     )

Commit message: Standarization
Parts:
- L1: footprint Tales:L_3x3_H1.5 -> Tales:L_3x3_h1.5
- L2: footprint Tales:L_12x12mm_H6mm -> Tales:L_12x12mm_h6mm
Changed lines of the file:
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@@
       (effects (font (size 1.27 1.27)))
     )
-    (property "Footprint" "Tales:L_12x12mm_H6mm" (at 196.85 46.99 0)
+    (property "Footprint" "Tales:L_12x12mm_h6mm" (at 196.85 46.99 0)
       (effects (font (size 1.27 1.27)) hide)
     )
@@
       (effects (font (size 1.27 1.27)))
     )
-    (property "Footprint" "Tales:L_3x3_H1.5" (at 68.58 124.46 0)
-      (effects (font (size 1.27 1.27)) hide)
-    )
+    (property "Footprint" "Tales:L_3x3_h1.5" (at 68.58 124.46 0)
+      (effects (font (size 1.27 1.27)) hide)
+    )
