File: V1/ESP-24v-32ch-V1.kicad_sch (KiCad schematic)
At the start: 8 parts, among them J1 Conn_01x08, J2 Conn_01x08, J3 Conn_01x08, J4 Conn_01x08, J5 Conn_01x08, J6 Conn_01x08, J7 Conn_01x08, J8 Conn_01x08

Commit message: Project rename
Other:
- sheet GPIO Expanders: file ESP-relay-32ch-V1-expanders.kicad_sch -> ESP-24v-32ch-V1-expanders.kicad_sch
- sheet Inputs 1-16: file ESP-relay-32ch-V1-inputs-1.kicad_sch -> ESP-24v-32ch-V1-inputs-1.kicad_sch
- sheet Inputs 17-32: file ESP-relay-32ch-V1-inputs-2.kicad_sch -> ESP-24v-32ch-V1-inputs-2.kicad_sch
- sheet LAN: file ESP-relay-32ch-V1-lan.kicad_sch -> ESP-24v-32ch-V1-lan.kicad_sch
- sheet MCU: file ESP-relay-32ch-V1-mcu.kicad_sch -> ESP-24v-32ch-V1-mcu.kicad_sch
- sheet Outputs 1-16: file ESP-relay-32ch-V1-outputs-1.kicad_sch -> ESP-24v-32ch-V1-outputs-1.kicad_sch
- sheet Outputs 17-32: file ESP-relay-32ch-V1-outputs-2.kicad_sch -> ESP-24v-32ch-V1-outputs-2.kicad_sch
- sheet Power: file ESP-relay-32ch-V1-power.kicad_sch -> ESP-24v-32ch-V1-power.kicad_sch
- title: ESP 32x 24VDC Input 32x External Relay Output Module -> ESP 32x 24VDC Input 32x 24VDC Output Module
Changed lines of the file:
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@@
   (paper "A4")
   (title_block
-    (title "ESP 32x 24VDC Input 32x External Relay Output Module")
-    (date "2023-04-24")
+    (title "ESP 32x 24VDC Input 32x 24VDC Output Module")
+    (date "2023-05-04")
     (rev "V1")
   )
@@
     (pin "8")
     (instances
-      (project "ESP-relay-32ch-V1"
+      (project "ESP-24v-32ch-V1"
         (path "/2bc5a21a-1d79-419d-a592-6852cc07b00a"
           (reference "J6") (unit 1)
@@
     (pin "8")
     (instances
-      (project "ESP-relay-32ch-V1"
+      (project "ESP-24v-32ch-V1"
         (path "/2bc5a21a-1d79-419d-a592-6852cc07b00a"
           (reference "J7") (unit 1)
@@
     (pin "8")
     (instances
-      (project "ESP-relay-32ch-V1"
+      (project "ESP-24v-32ch-V1"
         (path "/2bc5a21a-1d79-419d-a592-6852cc07b00a"
           (reference "J5") (unit 1)
@@
     (pin "8")
     (instances
-      (project "ESP-relay-32ch-V1"
+      (project "ESP-24v-32ch-V1"
         (path "/2bc5a21a-1d79-419d-a592-6852cc07b00a"
           (reference "J2") (unit 1)
@@
     (pin "8")
     (instances
-      (project "ESP-relay-32ch-V1"
+      (project "ESP-24v-32ch-V1"
         (path "/2bc5a21a-1d79-419d-a592-6852cc07b00a"
           (reference "J1") (unit 1)
@@
     (pin "8")
     (instances
-      (project "ESP-relay-32ch-V1"
+      (project "ESP-24v-32ch-V1"
         (path "/2bc5a21a-1d79-419d-a592-6852cc07b00a"
           (reference "J8") (unit 1)
@@
     (pin "8")
     (instances
-      (project "ESP-relay-32ch-V1"
+      (project "ESP-24v-32ch-V1"
         (path "/2bc5a21a-1d79-419d-a592-6852cc07b00a"
           (reference "J3") (unit 1)
@@
     (pin "8")
     (instances
-      (project "ESP-relay-32ch-V1"
+      (project "ESP-24v-32ch-V1"
         (path "/2bc5a21a-1d79-419d-a592-6852cc07b00a"
           (reference "J4") (unit 1)
@@
       (effects (font (size 1.27 1.27)) (justify left bottom))
     )
-    (property "Sheetfile" "ESP-relay-32ch-V1-inputs-2.kicad_sch" (at 60.96 155.5246 0)
+    (property "Sheetfile" "ESP-24v-32ch-V1-inputs-2.kicad_sch" (at 60.96 155.5246 0)
       (effects (font (size 1.27 1.27)) (justify left top))
     )
@@
     )
     (instances
-      (project "ESP-relay-32ch-V1"
+      (project "ESP-24v-32ch-V1"
         (path "/2bc5a21a-1d79-419d-a592-6852cc07b00a" (page "7"))
       )
@@
       (effects (font (size 1.27 1.27)) (justify left bottom))
     )
-    (property "Sheetfile" "ESP-relay-32ch-V1-outputs-1.kicad_sch" (at 198.12 104.7246 0)
+    (property "Sheetfile" "ESP-24v-32ch-V1-outputs-1.kicad_sch" (at 198.12 104.7246 0)
       (effects (font (size 1.27 1.27)) (justify left top))
     )
@@
     )
     (instances
-      (project "ESP-relay-32ch-V1"
+      (project "ESP-24v-32ch-V1"
         (path "/2bc5a21a-1d79-419d-a592-6852cc07b00a" (page "8"))
       )
@@
       (effects (font (size 1.27 1.27)) (justify left bottom))
     )
-    (property "Sheetfile" "ESP-relay-32ch-V1-power.kicad_sch" (at 60.96 36.1446 0)
+    (property "Sheetfile" "ESP-24v-32ch-V1-power.kicad_sch" (at 60.96 36.1446 0)
       (effects (font (size 1.27 1.27)) (justify left top))
     )
@@
     )
     (instances
-      (project "ESP-relay-32ch-V1"
+      (project "ESP-24v-32ch-V1"
         (path "/2bc5a21a-1d79-419d-a592-6852cc07b00a" (page "2"))
       )
@@
       (effects (font (size 1.27 1.27)) (justify left bottom))
     )
-    (property "Sheetfile" "ESP-relay-32ch-V1-inputs-1.kicad_sch" (at 60.96 104.7246 0)
+    (property "Sheetfile" "ESP-24v-32ch-V1-inputs-1.kicad_sch" (at 60.96 104.7246 0)
       (effects (font (size 1.27 1.27)) (justify left top))
     )
@@
     )
     (instances
-      (project "ESP-relay-32ch-V1"
+      (project "ESP-24v-32ch-V1"
         (path "/2bc5a21a-1d79-419d-a592-6852cc07b00a" (page "6"))
       )
@@
       (effects (font (size 1.27 1.27)) (justify left bottom))
     )
-    (property "Sheetfile" "ESP-relay-32ch-V1-expanders.kicad_sch" (at 109.22 155.5246 0)
+    (property "Sheetfile" "ESP-24v-32ch-V1-expanders.kicad_sch" (at 109.22 155.5246 0)
       (effects (font (size 1.27 1.27)) (justify left top))
     )
@@
     )
     (instances
-      (project "ESP-relay-32ch-V1"
+      (project "ESP-24v-32ch-V1"
         (path "/2bc5a21a-1d79-419d-a592-6852cc07b00a" (page "5"))
       )
@@
       (effects (font (size 1.27 1.27)) (justify left bottom))
     )
-    (property "Sheetfile" "ESP-relay-32ch-V1-lan.kicad_sch" (at 198.12 51.3846 0)
+    (property "Sheetfile" "ESP-24v-32ch-V1-lan.kicad_sch" (at 198.12 51.3846 0)
       (effects (font (size 1.27 1.27)) (justify left top))
     )
@@
     )
     (instances
-      (project "ESP-relay-32ch-V1"
+      (project "ESP-24v-32ch-V1"
         (path "/2bc5a21a-1d79-419d-a592-6852cc07b00a" (page "4"))
       )
@@
       (effects (font (size 1.27 1.27)) (justify left bottom))
     )
-    (property "Sheetfile" "ESP-relay-32ch-V1-outputs-2.kicad_sch" (at 198.12 155.5246 0)
+    (property "Sheetfile" "ESP-24v-32ch-V1-outputs-2.kicad_sch" (at 198.12 155.5246 0)
       (effects (font (size 1.27 1.27)) (justify left top))
     )
@@
     )
     (instances
-      (project "ESP-relay-32ch-V1"
+      (project "ESP-24v-32ch-V1"
         (path "/2bc5a21a-1d79-419d-a592-6852cc07b00a" (page "9"))
       )
@@
       (effects (font (size 1.27 1.27)) (justify left bottom))
     )
-    (property "Sheetfile" "ESP-relay-32ch-V1-mcu.kicad_sch" (at 109.22 51.3846 0)
+    (property "Sheetfile" "ESP-24v-32ch-V1-mcu.kicad_sch" (at 109.22 51.3846 0)
       (effects (font (size 1.27 1.27)) (justify left top))
     )
@@
     )
     (instances
-      (project "ESP-relay-32ch-V1"
+      (project "ESP-24v-32ch-V1"
         (path "/2bc5a21a-1d79-419d-a592-6852cc07b00a" (page "3"))
       )

Commit message: Replaced connector footprints
Parts:
- J1, J2, J3, J4, J5, J6, J7, J8: footprint Tales:TerminalBlock_Dorabo_DB141V-2.54-08P_1x08_P2.54mm_Vertical -> Tales:TerminalBlock_DG141V-2.54-8P_1x08_P2.54mm_Vertical
Changed lines of the file:
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@@
       (effects (font (size 1.27 1.27)))
     )
-    (property "Footprint" "Tales:TerminalBlock_Dorabo_DB141V-2.54-08P_1x08_P2.54mm_Vertical" (at 251.46 91.44 0)
+    (property "Footprint" "Tales:TerminalBlock_DG141V-2.54-8P_1x08_P2.54mm_Vertical" (at 251.46 91.44 0)
       (effects (font (size 1.27 1.27)) hide)
     )
@@
       (effects (font (size 1.27 1.27)))
     )
-    (property "Footprint" "Tales:TerminalBlock_Dorabo_DB141V-2.54-08P_1x08_P2.54mm_Vertical" (at 251.46 121.92 0)
+    (property "Footprint" "Tales:TerminalBlock_DG141V-2.54-8P_1x08_P2.54mm_Vertical" (at 251.46 121.92 0)
       (effects (font (size 1.27 1.27)) hide)
     )
@@
       (effects (font (size 1.27 1.27)))
     )
-    (property "Footprint" "Tales:TerminalBlock_Dorabo_DB141V-2.54-08P_1x08_P2.54mm_Vertical" (at 251.46 71.12 0)
+    (property "Footprint" "Tales:TerminalBlock_DG141V-2.54-8P_1x08_P2.54mm_Vertical" (at 251.46 71.12 0)
       (effects (font (size 1.27 1.27)) hide)
     )
@@
       (effects (font (size 1.27 1.27)))
     )
-    (property "Footprint" "Tales:TerminalBlock_Dorabo_DB141V-2.54-08P_1x08_P2.54mm_Vertical" (at 38.1 91.44 0)
+    (property "Footprint" "Tales:TerminalBlock_DG141V-2.54-8P_1x08_P2.54mm_Vertical" (at 38.1 91.44 0)
       (effects (font (size 1.27 1.27)) hide)
     )
@@
       (effects (font (size 1.27 1.27)))
     )
-    (property "Footprint" "Tales:TerminalBlock_Dorabo_DB141V-2.54-08P_1x08_P2.54mm_Vertical" (at 38.1 71.12 0)
+    (property "Footprint" "Tales:TerminalBlock_DG141V-2.54-8P_1x08_P2.54mm_Vertical" (at 38.1 71.12 0)
       (effects (font (size 1.27 1.27)) hide)
     )
@@
       (effects (font (size 1.27 1.27)))
     )
-    (property "Footprint" "Tales:TerminalBlock_Dorabo_DB141V-2.54-08P_1x08_P2.54mm_Vertical" (at 251.46 142.24 0)
+    (property "Footprint" "Tales:TerminalBlock_DG141V-2.54-8P_1x08_P2.54mm_Vertical" (at 251.46 142.24 0)
       (effects (font (size 1.27 1.27)) hide)
     )
@@
       (effects (font (size 1.27 1.27)))
     )
-    (property "Footprint" "Tales:TerminalBlock_Dorabo_DB141V-2.54-08P_1x08_P2.54mm_Vertical" (at 38.1 121.92 0)
+    (property "Footprint" "Tales:TerminalBlock_DG141V-2.54-8P_1x08_P2.54mm_Vertical" (at 38.1 121.92 0)
       (effects (font (size 1.27 1.27)) hide)
     )
@@
       (effects (font (size 1.27 1.27)))
     )
-    (property "Footprint" "Tales:TerminalBlock_Dorabo_DB141V-2.54-08P_1x08_P2.54mm_Vertical" (at 38.1 142.24 0)
-      (effects (font (size 1.27 1.27)) hide)
-    )
+    (property "Footprint" "Tales:TerminalBlock_DG141V-2.54-8P_1x08_P2.54mm_Vertical" (at 38.1 142.24 0)
+      (effects (font (size 1.27 1.27)) hide)
+    )

Commit message: Connectors rotated 180deg
Other:
- note added: "UPDATES PARA V2: ALTERAR CONECTOR USB PARA 2.0 TIPO C HORIZONTAL ALTERAR CONECTOR 24V PARA SPRING CAGE ADICIONAR POE MOVER LED POWER PARA RAIL 5V REFAZER LAYOUT EM 4 LAYERS PARA DIMINUIR TAMANHO"
Changed lines of the file:
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@@
     (stroke (width 0) (type default))
+  )
+  (text "UPDATES PARA V2:\nALTERAR CONECTOR USB PARA 2.0 TIPO C HORIZONTAL\nALTERAR CONECTOR 24V PARA SPRING CAGE\nADICIONAR POE\nMOVER LED POWER PARA RAIL 5V\nREFAZER LAYOUT EM 4 LAYERS PARA DIMINUIR TAMANHO"
+    (at 60.96 187.96 0)
+    (effects (font (size 2.54 2.54)) (justify left bottom))
   )
   (symbol (lib_id "Connector_Generic:Conn_01x08") (at 251.46 91.44 0) (unit 1)

Commit message: Design optimization
Parts:
- J1, J2, J3, J4, J5, J6, J7, J8: value Conn_01x08 -> DB141V-2.54-8P; footprint Tales:TerminalBlock_DG141V-2.54-8P_1x08_P2.54mm_Vertical -> Tales:TerminalBlock_Dibo_DB141V-2.54-8P_1x08_P2.54mm_Vertical
Changed lines of the file:
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@@
       (effects (font (size 1.27 1.27)))
     )
-    (property "Value" "Conn_01x08" (at 261.62 91.44 0)
-      (effects (font (size 1.27 1.27)))
-    )
-    (property "Footprint" "Tales:TerminalBlock_DG141V-2.54-8P_1x08_P2.54mm_Vertical" (at 251.46 91.44 0)
+    (property "Value" "DB141V-2.54-8P" (at 261.62 91.44 0)
+      (effects (font (size 1.27 1.27)))
+    )
+    (property "Footprint" "Tales:TerminalBlock_Dibo_DB141V-2.54-8P_1x08_P2.54mm_Vertical" (at 251.46 91.44 0)
       (effects (font (size 1.27 1.27)) hide)
     )
@@
       (effects (font (size 1.27 1.27)))
     )
-    (property "Value" "Conn_01x08" (at 261.62 121.92 0)
-      (effects (font (size 1.27 1.27)))
-    )
-    (property "Footprint" "Tales:TerminalBlock_DG141V-2.54-8P_1x08_P2.54mm_Vertical" (at 251.46 121.92 0)
+    (property "Value" "DB141V-2.54-8P" (at 261.62 121.92 0)
+      (effects (font (size 1.27 1.27)))
+    )
+    (property "Footprint" "Tales:TerminalBlock_Dibo_DB141V-2.54-8P_1x08_P2.54mm_Vertical" (at 251.46 121.92 0)
       (effects (font (size 1.27 1.27)) hide)
     )
@@
       (effects (font (size 1.27 1.27)))
     )
-    (property "Value" "Conn_01x08" (at 261.62 71.12 0)
-      (effects (font (size 1.27 1.27)))
-    )
-    (property "Footprint" "Tales:TerminalBlock_DG141V-2.54-8P_1x08_P2.54mm_Vertical" (at 251.46 71.12 0)
+    (property "Value" "DB141V-2.54-8P" (at 261.62 71.12 0)
+      (effects (font (size 1.27 1.27)))
+    )
+    (property "Footprint" "Tales:TerminalBlock_Dibo_DB141V-2.54-8P_1x08_P2.54mm_Vertical" (at 251.46 71.12 0)
       (effects (font (size 1.27 1.27)) hide)
     )
@@
       (effects (font (size 1.27 1.27)))
     )
-    (property "Value" "Conn_01x08" (at 27.94 91.44 0)
-      (effects (font (size 1.27 1.27)))
-    )
-    (property "Footprint" "Tales:TerminalBlock_DG141V-2.54-8P_1x08_P2.54mm_Vertical" (at 38.1 91.44 0)
+    (property "Value" "DB141V-2.54-8P" (at 27.94 91.44 0)
+      (effects (font (size 1.27 1.27)))
+    )
+    (property "Footprint" "Tales:TerminalBlock_Dibo_DB141V-2.54-8P_1x08_P2.54mm_Vertical" (at 38.1 91.44 0)
       (effects (font (size 1.27 1.27)) hide)
     )
@@
       (effects (font (size 1.27 1.27)))
     )
-    (property "Value" "Conn_01x08" (at 27.94 71.12 0)
-      (effects (font (size 1.27 1.27)))
-    )
-    (property "Footprint" "Tales:TerminalBlock_DG141V-2.54-8P_1x08_P2.54mm_Vertical" (at 38.1 71.12 0)
+    (property "Value" "DB141V-2.54-8P" (at 27.94 71.12 0)
+      (effects (font (size 1.27 1.27)))
+    )
+    (property "Footprint" "Tales:TerminalBlock_Dibo_DB141V-2.54-8P_1x08_P2.54mm_Vertical" (at 38.1 71.12 0)
       (effects (font (size 1.27 1.27)) hide)
     )
@@
       (effects (font (size 1.27 1.27)))
     )
-    (property "Value" "Conn_01x08" (at 261.62 142.24 0)
-      (effects (font (size 1.27 1.27)))
-    )
-    (property "Footprint" "Tales:TerminalBlock_DG141V-2.54-8P_1x08_P2.54mm_Vertical" (at 251.46 142.24 0)
+    (property "Value" "DB141V-2.54-8P" (at 261.62 142.24 0)
+      (effects (font (size 1.27 1.27)))
+    )
+    (property "Footprint" "Tales:TerminalBlock_Dibo_DB141V-2.54-8P_1x08_P2.54mm_Vertical" (at 251.46 142.24 0)
       (effects (font (size 1.27 1.27)) hide)
     )
@@
       (effects (font (size 1.27 1.27)))
     )
-    (property "Value" "Conn_01x08" (at 27.94 121.92 0)
-      (effects (font (size 1.27 1.27)))
-    )
-    (property "Footprint" "Tales:TerminalBlock_DG141V-2.54-8P_1x08_P2.54mm_Vertical" (at 38.1 121.92 0)
+    (property "Value" "DB141V-2.54-8P" (at 27.94 121.92 0)
+      (effects (font (size 1.27 1.27)))
+    )
+    (property "Footprint" "Tales:TerminalBlock_Dibo_DB141V-2.54-8P_1x08_P2.54mm_Vertical" (at 38.1 121.92 0)
       (effects (font (size 1.27 1.27)) hide)
     )
@@
       (effects (font (size 1.27 1.27)))
     )
-    (property "Value" "Conn_01x08" (at 27.94 142.24 0)
-      (effects (font (size 1.27 1.27)))
-    )
-    (property "Footprint" "Tales:TerminalBlock_DG141V-2.54-8P_1x08_P2.54mm_Vertical" (at 38.1 142.24 0)
-      (effects (font (size 1.27 1.27)) hide)
-    )
+    (property "Value" "DB141V-2.54-8P" (at 27.94 142.24 0)
+      (effects (font (size 1.27 1.27)))
+    )
+    (property "Footprint" "Tales:TerminalBlock_Dibo_DB141V-2.54-8P_1x08_P2.54mm_Vertical" (at 38.1 142.24 0)
+      (effects (font (size 1.27 1.27)) hide)
+    )
